Commit message: restructed into macros and exposed com port

File: ewellix_liftkit_description/urdf/ewellix_liftkit.ros2_control.xacro (robot description, xacro)
@@ -1,27 +1,29 @@
 <?xml version="1.0"?>
 <robot xmlns:xacro="http://www.ros.org/wiki/xacro">
-  <xacro:macro name="robotiq_gripper_ros2_control" params="
-        name:=liftkit_ros2_control
-        prefix
-        use_fake_hardware:=false
-        com_port:=/dev/ttyUSB0
-        baudrate:=34800">
-  <ros2_control name="${name}" type="actuator">
-    <hardware>
-      <xacro:if value="${use_fake_hardware}">
-        <plugin>mock_components/GenericSystem</plugin>
-      </xacro:if>
-      <xacro:unless value="${use_fake_hardware}">
-        <plugin>liftkit_hardware_interface/LiftkitHardwareInterface</plugin>
-        <param name="lift_name">liftkit</param>
-        <param name="COM_port">${com_port}</param>
-        <param name="baudrate">${baudrate}</param>
-      </xacro:unless>
-    </hardware>
-    <joint name=">${prefix}ewellix_lift_top_joint">
-      <command_interface name="position"/>
-      <state_interface name="position"/>
-      <state_interface name="velocity"/>
-      <state_interface name="robot_ready"/>
-    </joint>
-  </ros2_control>
+  <xacro:macro name="ewellix_liftkit_ros2_control" params="
+    name
+    tf_prefix
+    use_fake_hardware:=false
+    com_port:=/dev/ttyUSB0
+    baudrate:=34800">
+    <ros2_control name="${name}" type="actuator">
+      <hardware>
+        <xacro:if value="${use_fake_hardware}">
+          <plugin>mock_components/GenericSystem</plugin>
+        </xacro:if>
+        <xacro:unless value="${use_fake_hardware}">
+          <plugin>liftkit_hardware_interface/LiftkitHardwareInterface</plugin>
+          <param name="lift_name">liftkit</param>
+          <param name="COM_port">${com_port}</param>
+          <param name="baudrate">${baudrate}</param>
+        </xacro:unless>
+      </hardware>
+      <joint name=">${tf_prefix}ewellix_lift_top_joint">
+        <command_interface name="position"/>
+        <state_interface name="position"/>
+        <state_interface name="velocity"/>
+        <state_interface name="robot_ready"/>
+      </joint>
+    </ros2_control>
+  </xacro:macro>
+</robot>

File: ewellix_liftkit_description/urdf/ewellix_macro.urdf.xacro (robot description, xacro)
@@ -1,49 +1,66 @@
 <?xml version="1.0"?>
-<robot name="ewellix_lift_700mm" xmlns:xacro="http://www.ros.org/wiki/xacro">
-<!-- TODO turn this into a macro-->
-<xacro:property name="M_PI" value="3.1415926535897931" />
-  <link name="ewellix_lift_base_link">
-    <visual>
-      <origin xyz="0 0 0" rpy="0 0 0"/>
-      <geometry>
-        <mesh filename="file://$(find ewellix_liftkit_description)/meshes/visual/ewellix_lift_base_700mm.stl"/>
-      </geometry>
-      <material name="grey">
-        <color rgba="0.7 0.7 0.7 1"/>
-      </material>
-    </visual>
-    <collision>
-      <origin xyz="-0.005 0 0.00235" rpy="0 0 0"/>
-      <geometry>
-        <mesh filename="file://$(find ewellix_liftkit_description)/meshes/visual/ewellix_lift_base_700mm.stl"/>
-      </geometry>
-    </collision>
-  </link>
-  <!-- Lift top link -->
-  <link name="ewellix_lift_top_link">
-    <visual>
-      <origin xyz="0 0 0" rpy="0 0 0"/>
-      <geometry>
-        <mesh filename="file://$(find ewellix_liftkit_description)/meshes/visual/ewellix_lift_top_700mm.stl"/>
-      </geometry>
-      <material name="grey">
-        <color rgba="0.7 0.7 0.7 1"/>
-      </material>
-    </visual>
-    <!-- TODO figure out how to retract the top link entirely without it colliding through the base. Consider splitting the top into two pieces with a mimic joint-->
-    <collision>
-      <origin xyz="-0.005 0 0.00235" rpy="0 0 0"/>
-      <geometry>
-        <mesh filename="file://$(find ewellix_liftkit_description)/meshes/visual/ewellix_lift_top_700mm.stl"/>
-      </geometry>
-    </collision>
-  </link>
-  <!-- Lift top link joint -->
-  <joint name="ewellix_lift_top_joint" type="prismatic">
-    <parent link="ewellix_lift_base_link"/>
-    <child link="ewellix_lift_top_link" />
-    <origin xyz="0 0 0.730" rpy="0 0 0" />
-    <limit effort="1000" lower="0.0" upper="0.7" velocity="0.088"/>
-    <axis xyz="0 0 1" />
-  </joint>
+<robot xmlns:xacro="http://www.ros.org/wiki/xacro">
+  <xacro:property name="M_PI" value="3.1415926535897931" />
+  <xacro:macro name="ewellix_lift" params="
+    name
+    tf_prefix
+    use_fake_hardware:=false
+    com_port:=/dev/ttyUSB0
+    baudrate:=34800
+  ">
+    <!-- TODO work on abstracting this xacro to work for both 500 and 700mm lifts -->
+    <link name="${tf_prefix}ewellix_lift_base_link">
+      <visual>
+        <origin xyz="0 0 0" rpy="0 0 0"/>
+        <geometry>
+          <mesh filename="file://$(find ewellix_liftkit_description)/meshes/visual/ewellix_lift_base_700mm.stl"/>
+        </geometry>
+        <material name="grey">
+          <color rgba="0.7 0.7 0.7 1"/>
+        </material>
+      </visual>
+      <!-- TODO is this a good collision?-->
+      <collision>
+        <origin xyz="-0.005 0 0.00235" rpy="0 0 0"/>
+        <geometry>
+          <mesh filename="file://$(find ewellix_liftkit_description)/meshes/visual/ewellix_lift_base_700mm.stl"/>
+        </geometry>
+      </collision>
+    </link>
+    <!-- Lift top link -->
+    <link name="${tf_prefix}ewellix_lift_top_link">
+      <visual>
+        <origin xyz="0 0 0" rpy="0 0 0"/>
+        <geometry>
+          <mesh filename="file://$(find ewellix_liftkit_description)/meshes/visual/ewellix_lift_top_700mm.stl"/>
+        </geometry>
+        <material name="grey">
+          <color rgba="0.7 0.7 0.7 1"/>
+        </material>
+      </visual>
+      <!-- TODO figure out how to retract the top link entirely without it colliding through the base. Consider splitting the top into two pieces with a mimic joint-->
+      <collision>
+        <origin xyz="-0.005 0 0.00235" rpy="0 0 0"/>
+        <geometry>
+          <mesh filename="file://$(find ewellix_liftkit_description)/meshes/visual/ewellix_lift_top_700mm.stl"/>
+        </geometry>
+      </collision>
+    </link>
+    <!-- Lift top link joint -->
+    <joint name="${tf_prefix}ewellix_lift_top_joint" type="prismatic">
+      <parent link="${tf_prefix}ewellix_lift_base_link"/>
+      <child link="${tf_prefix}ewellix_lift_top_link" />
+      <origin xyz="0 0 0.730" rpy="0 0 0" />
+      <limit effort="1000" lower="0.0" upper="0.7" velocity="0.088"/>
+      <axis xyz="0 0 1" />
+    </joint>
+    <xacro:include filename="$(find ewellix_liftkit_description)/urdf/ewellix_liftkit.ros2_control.xacro" />
+    <xacro:ewellix_liftkit_ros2_control
+      name="${name}"
+      use_fake_hardware="${use_fake_hardware}"
+      tf_prefix="${tf_prefix}"
+      com_port="${com_port}"
+      baudrate="${baudrate}"
+    />
+  </xacro:macro>
 </robot>

Commit message: reworked to get fake hardware working

File: ewellix_liftkit_description/urdf/ewellix_liftkit.ros2_control.xacro (robot description, xacro)
@@ -7,23 +7,36 @@
     com_port:=/dev/ttyUSB0
     baudrate:=34800">
-    <ros2_control name="${name}" type="actuator">
-      <hardware>
-        <xacro:if value="${use_fake_hardware}">
-          <plugin>mock_components/GenericSystem</plugin>
-        </xacro:if>
-        <xacro:unless value="${use_fake_hardware}">
-          <plugin>liftkit_hardware_interface/LiftkitHardwareInterface</plugin>
-          <param name="lift_name">liftkit</param>
-          <param name="COM_port">${com_port}</param>
-          <param name="baudrate">${baudrate}</param>
-        </xacro:unless>
-      </hardware>
-      <joint name=">${tf_prefix}ewellix_lift_top_joint">
-        <command_interface name="position"/>
-        <state_interface name="position"/>
-        <state_interface name="velocity"/>
-        <state_interface name="robot_ready"/>
-      </joint>
-    </ros2_control>
+    <xacro:unless value="${use_fake_hardware}">
+      <ros2_control name="${name}" type="actuator">
+        <hardware>
+            <plugin>liftkit_hardware_interface/LiftkitHardwareInterface</plugin>
+            <param name="lift_name">liftkit</param>
+            <param name="COM_port">${com_port}</param>
+            <param name="baudrate">${baudrate}</param>
+        </hardware>
+        <joint name="${tf_prefix}ewellix_lift_top_joint">
+          <command_interface name="position"/>
+          <state_interface name="position"/>
+          <state_interface name="velocity"/>
+          <state_interface name="robot_ready"/>
+        </joint>
+      </ros2_control>
+    </xacro:unless>
+    <xacro:if value="${use_fake_hardware}">
+      <ros2_control name="${name}" type="system">
+        <hardware>
+            <plugin>mock_components/GenericSystem</plugin>
+        </hardware>
+        <joint name="${tf_prefix}ewellix_lift_top_joint">
+          <command_interface name="position">
+            <param name="min">0</param>
+            <param name="max">0.7</param>
+          </command_interface>
+          <state_interface name="position"/>
+          <state_interface name="velocity"/>
+          <state_interface name="robot_ready"/>
+        </joint>
+      </ros2_control>
+    </xacro:if>
   </xacro:macro>
 </robot>
