Commit message: restructing to macros

File: ewellix_liftkit_description/urdf/ewellix_macro.urdf.xacro (robot description, xacro)
@@ -47,16 +47,3 @@
     <axis xyz="0 0 1" />
   </joint>
-  <!-- TODO add in fake hardware -->
-  <ros2_control name="liftkit_ros2_control" type="actuator">
-      <hardware>
-          <plugin>liftkit_hardware_interface/LiftkitHardwareInterface</plugin>
-          <param name="lift_name">liftkit</param>
-      </hardware>
-      <joint name="ewellix_lift_top_joint">
-          <command_interface name="position"/>
-          <state_interface name="position"/>
-          <state_interface name="velocity"/>
-          <state_interface name="robot_ready"/>
-      </joint>
-  </ros2_control>
 </robot>

Commit message: Adjusted to include parent link for base

File: ewellix_liftkit_description/urdf/ewellix_macro.urdf.xacro (robot description, xacro)
@@ -5,4 +5,5 @@
     name
     tf_prefix
+    parent
     use_fake_hardware:=false
     com_port:=/dev/ttyUSB0
@@ -47,4 +48,10 @@
       </collision>
     </link>
+    <!-- Lift base link joint -->
+    <joint name="${tf_prefix}ewellix_lift_base_joint" type="fixed">
+      <parent link="${parent}"/>
+      <child link="${tf_prefix}ewellix_lift_base_link" />
+      <origin xyz="-0.1115 0.0 0.0565" rpy="0 0 3.14159"/>
+    </joint>
     <!-- Lift top link joint -->
     <joint name="${tf_prefix}ewellix_lift_top_joint" type="prismatic">

Commit message: updating meshes and developing ewellix_macro.urdf.xacro using fixed links, need more fixed links, collision primatives, and inertial data, NOT WORKING

File: ewellix_liftkit_description/urdf/ewellix_macro.urdf.xacro (robot description, xacro)
@@ -9,50 +9,107 @@
     baudrate:=34800
   ">
-    <!-- TODO work on abstracting this xacro to work for both 500 and 700mm lifts -->
+    <!-- TODO work on abstracting this xacro to work for both 500 and 700mm lifts (I'll give it a shot -Mike)-->
+    <!-- TODO is this a good collision? (No, it wasn't, raw meshes in general do not make good collision objects -Mike)-->
+    <!-- TODO figure out how to retract the top link entirely without it colliding through the base. Consider splitting the top into two pieces with a mimic joint (Will do -Mike)-->
+    <!-- Sure hope this is all works in SI units... -Mike-->
+    <!--BASE-->
     <link name="${tf_prefix}ewellix_lift_base_link">
+      <inertia>
+        <mass value="1.7383784"/>
+        <inertia ixx="5.7788770e-03" ixy="0" ixz="0" iyy="7.0031715e-03" iyz="0" izz="1.2717018e-02"/>
+      </inertia>
       <visual>
-        <origin xyz="0 0 0" rpy="0 0 0"/>
         <geometry>
-          <mesh filename="file://$(find ewellix_liftkit_description)/meshes/visual/ewellix_lift_base_700mm.stl"/>
+          <box size="0.220 0.200 0.015"/>
         </geometry>
-        <material name="grey">
-          <color rgba="0.7 0.7 0.7 1"/>
-        </material>
       </visual>
-      <!-- TODO is this a good collision?-->
       <collision>
-        <origin xyz="-0.005 0 0.00235" rpy="0 0 0"/>
         <geometry>
-          <mesh filename="file://$(find ewellix_liftkit_description)/meshes/visual/ewellix_lift_base_700mm.stl"/>
+          <box size="0.220 0.200 0.015"/>
         </geometry>
       </collision>
     </link>
-    <!-- Lift top link -->
-    <link name="${tf_prefix}ewellix_lift_top_link">
+    <!--LOWER-->
+    <link name="${tf_prefix}ewellix_lift_lower_link">
+      <!-- TODO -Mike
+      <inertia>
+        <mass value=""/>
+        <inertia ixx="" ixy="" ixz="" iyy="" iyz="" izz=""/>
+      </inertia>
+      -->
       <visual>
-        <origin xyz="0 0 0" rpy="0 0 0"/>
         <geometry>
-          <mesh filename="file://$(find ewellix_liftkit_description)/meshes/visual/ewellix_lift_top_700mm.stl"/>
+          <mesh filename= "file://$(find ewellix_liftkit_description)/meshes/visual/lift_low.dae"/>
         </geometry>
-        <material name="grey">
-          <color rgba="0.7 0.7 0.7 1"/>
-        </material>
       </visual>
-      <!-- TODO figure out how to retract the top link entirely without it colliding through the base. Consider splitting the top into two pieces with a mimic joint-->
       <collision>
-        <origin xyz="-0.005 0 0.00235" rpy="0 0 0"/>
         <geometry>
-          <mesh filename="file://$(find ewellix_liftkit_description)/meshes/visual/ewellix_lift_top_700mm.stl"/>
+          <box size="0.163 0.163 0.480"/>
         </geometry>
       </collision>
     </link>
-    <!-- Lift top link joint -->
-    <joint name="${tf_prefix}ewellix_lift_top_joint" type="prismatic">
+    <!--BASE TO LOWER-->
+    <joint name="base_to_lower" type="fixed">
       <parent link="${tf_prefix}ewellix_lift_base_link"/>
-      <child link="${tf_prefix}ewellix_lift_top_link" />
-      <origin xyz="0 0 0.730" rpy="0 0 0" />
-      <limit effort="1000" lower="0.0" upper="0.7" velocity="0.088"/>
-      <axis xyz="0 0 1" />
+      <child link="${tf_prefix}ewellix_lift_lower_link"/>
+      <origin xyz="0 0 0.2475" rpy="0 0 0"/>
     </joint>
+    <!--MIDDLE-->
+    <link name="${tf_prefix}ewellix_lift_middle_link">
+      <!-- TODO -Mike
+      <inertia>
+        <mass value=""/>
+        <inertia ixx="" ixy="" ixz="" iyy="" iyz="" izz=""/>
+      </inertia>
+      -->
+      <visual>
+        <geometry>
+          <mesh filename= "file://$(find ewellix_liftkit_description)/meshes/visual/lift_mid.dae"/>
+        </geometry>
+      </visual>
+      <collision>
+        <geometry>
+          <box size="0.146 0.146 0.483"/>
+        </geometry>
+      </collision>
+    </link>
+    <!--HIGHER-->
+    <link name="${tf_prefix}ewellix_lift_higher_link">
+      <!-- TODO -Mike
+      <inertia>
+        <mass value=""/>
+        <inertia ixx="" ixy="" ixz="" iyy="" iyz="" izz=""/>
+      </inertia>
+      -->
+      <visual>
+        <geometry>
+          <mesh filename= "file://$(find ewellix_liftkit_description)/meshes/visual/lift_high.dae"/>
+        </geometry>
+      </visual>
+      <collision>
+        <geometry>
+          <box size="0.129 0.129 0.488"/>
+        </geometry>
+      </collision>
+    </link>
+    <!--TOP-->
+    <link name="${tf_prefix}ewellix_lift_top_link">
+      <!-- TODO -Mike
+      <inertia>
+        <mass value=""/>
+        <inertia ixx="" ixy="" ixz="" iyy="" iyz="" izz=""/>
+      </inertia>
+      -->
+      <visual>
+        <geometry>
+          <box size="0.200 0.220 0.015"/>
+        </geometry>
+      </visual>
+      <collision>
+        <geometry>
+          <box size="0.200 0.220 0.015"/>
+        </geometry>
+      </collision>
+    </link>
     <xacro:include filename="$(find ewellix_liftkit_description)/urdf/ewellix_liftkit.ros2_control.xacro" />
     <xacro:ewellix_liftkit_ros2_control

Commit message: description running with fixed joints, moving on to kinematic definitions

File: ewellix_liftkit_description/urdf/ewellix_macro.urdf.xacro (robot description, xacro)
@@ -93,4 +93,16 @@
       </collision>
     </link>
+    <!--LOWER TO HIGHER-->
+    <joint name="lower_to_higher" type="fixed">
+      <parent link="${tf_prefix}ewellix_lift_lower_link"/>
+      <child link="${tf_prefix}ewellix_lift_higher_link"/>
+      <origin xyz="0 0 0.0454" rpy="0 0 0"/>
+    </joint>
+    <!--MIDDLE MIMIC HIGHER-->
+    <joint name="middle_mimic_higher" type="fixed">
+      <parent link="${tf_prefix}ewellix_lift_higher_link"/>
+      <child link="${tf_prefix}ewellix_lift_middle_link"/>
+      <origin xyz="0 0 -0.0222" rpy="0 0 0"/>
+    </joint>
     <!--TOP-->
     <link name="${tf_prefix}ewellix_lift_top_link">
@@ -112,4 +124,10 @@
       </collision>
     </link>
+    <!--HIGHER TO TOP-->
+    <joint name="higher_to_top" type="fixed">
+      <parent link="${tf_prefix}ewellix_lift_higher_link"/>
+      <child link="${tf_prefix}ewellix_lift_top_link"/>
+      <origin xyz="0 0 0.2515" rpy="0 0 0"/>
+    </joint>
     <xacro:include filename="$(find ewellix_liftkit_description)/urdf/ewellix_liftkit.ros2_control.xacro" />
     <xacro:ewellix_liftkit_ros2_control

Commit message: added kinematic definitions, still need to add inertias and masses. Odd error 'Invalid frame ID' for the middle link?

File: ewellix_liftkit_description/urdf/ewellix_macro.urdf.xacro (robot description, xacro)
@@ -49,5 +49,5 @@
       </collision>
     </link>
-    <!--BASE TO LOWER-->
+    <!--BASE TO LOWER (FIXED)-->
     <joint name="base_to_lower" type="fixed">
       <parent link="${tf_prefix}ewellix_lift_base_link"/>
@@ -93,15 +93,20 @@
       </collision>
     </link>
-    <!--LOWER TO HIGHER-->
-    <joint name="lower_to_higher" type="fixed">
+    <!--LOWER TO HIGHER (PRIS)-->
+    <joint name="lower_to_higher" type="prismatic">
       <parent link="${tf_prefix}ewellix_lift_lower_link"/>
       <child link="${tf_prefix}ewellix_lift_higher_link"/>
       <origin xyz="0 0 0.0454" rpy="0 0 0"/>
+      <axis xyz="0 0 1"/>
+      <limit lower="0" upper="0.7" effort="1000" velocity="1"/>
     </joint>
-    <!--MIDDLE MIMIC HIGHER-->
-    <joint name="middle_mimic_higher" type="fixed">
+    <!--MIDDLE MIMIC HIGHER (PRIS MIMIC)-->
+    <joint name="middle_mimic_higher" type="prismatic">
       <parent link="${tf_prefix}ewellix_lift_higher_link"/>
       <child link="${tf_prefix}ewellix_lift_middle_link"/>
       <origin xyz="0 0 -0.0222" rpy="0 0 0"/>
+      <axis xyz="0 0 -1"/>
+      <limit lower="0" upper="0.351" effort="1000" velocity="1"/>
+      <mimic joint="lower_to_higher" multiplier="0.5" offset="0"/>
     </joint>
     <!--TOP-->
@@ -124,5 +129,5 @@
       </collision>
     </link>
-    <!--HIGHER TO TOP-->
+    <!--HIGHER TO TOP (FIXED)-->
     <joint name="higher_to_top" type="fixed">
       <parent link="${tf_prefix}ewellix_lift_higher_link"/>

Commit message: added inertial properties and recolored base and top links, ready for review

File: ewellix_liftkit_description/urdf/ewellix_macro.urdf.xacro (robot description, xacro)
@@ -23,4 +23,7 @@
           <box size="0.220 0.200 0.015"/>
         </geometry>
+        <material name="gray">
+          <color rgba="0.85 0.85 0.85 1"/>
+        </material>
       </visual>
       <collision>
@@ -32,10 +35,8 @@
     <!--LOWER-->
     <link name="${tf_prefix}ewellix_lift_lower_link">
-      <!-- TODO -Mike
       <inertia>
-        <mass value=""/>
-        <inertia ixx="" ixy="" ixz="" iyy="" iyz="" izz=""/>
+        <mass value="1.9521070e+01"/>
+        <inertia ixx="0.46604111" ixy="0" ixz="0" iyy="0.46480515" iyz="-0.002668667" izz="0.1561"/>
       </inertia>
-      -->
       <visual>
         <geometry>
@@ -57,10 +58,8 @@
     <!--MIDDLE-->
     <link name="${tf_prefix}ewellix_lift_middle_link">
-      <!-- TODO -Mike
       <inertia>
-        <mass value=""/>
-        <inertia ixx="" ixy="" ixz="" iyy="" iyz="" izz=""/>
+        <mass value="1.5593303e+01"/>
+        <inertia ixx="0.34930648" ixy="0" ixz="0" iyy="0.34930648" iyz="0" izz="0.095393471"/>
       </inertia>
-      -->
       <visual>
         <geometry>
@@ -76,10 +75,8 @@
     <!--HIGHER-->
     <link name="${tf_prefix}ewellix_lift_higher_link">
-      <!-- TODO -Mike
       <inertia>
-        <mass value=""/>
-        <inertia ixx="" ixy="" ixz="" iyy="" iyz="" izz=""/>
+        <mass value="1.5166778e+01"/>
+        <inertia ixx="0.35552099" ixy="9.6314989e-6" ixz="2.284786e-5" iyy="0.35552876" iyz="5.4910201e-5" izz="0.069925583"/>
       </inertia>
-      -->
       <visual>
         <geometry>
@@ -112,14 +109,15 @@
     <!--TOP-->
     <link name="${tf_prefix}ewellix_lift_top_link">
-      <!-- TODO -Mike
       <inertia>
-        <mass value=""/>
-        <inertia ixx="" ixy="" ixz="" iyy="" iyz="" izz=""/>
+        <mass value="4.9139525"/>
+        <inertia ixx="0.02015548" ixy="-2.281101e-5" ixz="0" iyy="0.01664141" iyz="0" izz="0.03661307"/>
       </inertia>
-      -->
       <visual>
         <geometry>
           <box size="0.200 0.220 0.015"/>
         </geometry>
+        <material name="gray">
+          <color rgba="0.85 0.85 0.85 1"/>
+        </material>
       </visual>
       <collision>
