Commit message: separated out description package

File: ewellix_liftkit_description/urdf/ewellix_lift_700mm.urdf.xacro (robot description, xacro)
@@ -1,4 +1,5 @@
 <?xml version="1.0"?>
 <robot name="ewellix_lift_700mm" xmlns:xacro="http://www.ros.org/wiki/xacro">
+<!-- TODO turn this into a macro-->
 <xacro:property name="M_PI" value="3.1415926535897931" />
   <link name="ewellix_lift_base_link">
@@ -6,5 +7,5 @@
       <origin xyz="0 0 0" rpy="0 0 0"/>
       <geometry>
-        <mesh filename="$(find liftkit)/meshes/ewellix_lift_base_700mm.stl"/>
+        <mesh filename="file://$(find ewellix_liftkit_description)/meshes/visual/ewellix_lift_base_700mm.stl"/>
       </geometry>
       <material name="grey">
@@ -15,32 +16,27 @@
       <origin xyz="-0.005 0 0.00235" rpy="0 0 0"/>
       <geometry>
-        <mesh filename="$(find liftkit)/meshes/ewellix_lift_base_700mm.stl"/>
+        <mesh filename="file://$(find ewellix_liftkit_description)/meshes/visual/ewellix_lift_base_700mm.stl"/>
       </geometry>
     </collision>
   </link>
-  <!-- Lift base link joint
-  <joint name="ewellix_lift_base_joint" type="fixed">
-    <xacro:insert_block name="origin" />
-    <parent link="${parent}"/>
-    <child link="ewellix_lift_base_link" />
-  </joint> -->
-    <!-- Lift top link -->
-    <link name="ewellix_lift_top_link">
-      <visual>
-        <origin xyz="0 0 0" rpy="0 0 0"/>
-        <geometry>
-          <mesh filename="$(find liftkit)/meshes/ewellix_lift_top_700mm.stl"/>
-        </geometry>
-        <material name="grey">
-          <color rgba="0.7 0.7 0.7 1"/>
-        </material>
-      </visual>
-      <collision>
-        <origin xyz="-0.005 0 0.00235" rpy="0 0 0"/>
-        <geometry>
-          <mesh filename="$(find liftkit)/meshes/ewellix_lift_top_700mm.stl"/>
-        </geometry>
-      </collision>
-    </link>
+  <!-- Lift top link -->
+  <link name="ewellix_lift_top_link">
+    <visual>
+      <origin xyz="0 0 0" rpy="0 0 0"/>
+      <geometry>
+        <mesh filename="file://$(find ewellix_liftkit_description)/meshes/visual/ewellix_lift_top_700mm.stl"/>
+      </geometry>
+      <material name="grey">
+        <color rgba="0.7 0.7 0.7 1"/>
+      </material>
+    </visual>
+    <!-- TODO figure out how to retract the top link entirely without it colliding through the base. Consider splitting the top into two pieces with a mimic joint-->
+    <collision>
+      <origin xyz="-0.005 0 0.00235" rpy="0 0 0"/>
+      <geometry>
+        <mesh filename="file://$(find ewellix_liftkit_description)/meshes/visual/ewellix_lift_top_700mm.stl"/>
+      </geometry>
+    </collision>
+  </link>
   <!-- Lift top link joint -->
   <joint name="ewellix_lift_top_joint" type="prismatic">
@@ -51,15 +47,9 @@
     <axis xyz="0 0 1" />
   </joint>
-  <!--
-      PositionJointInterface
-      VelocityJointInterface
-      EffortJointInterface
-  -->
+  <!-- TODO add in fake hardware -->
   <ros2_control name="liftkit_ros2_control" type="actuator">
       <hardware>
           <plugin>liftkit_hardware_interface/LiftkitHardwareInterface</plugin>
           <param name="lift_name">liftkit</param>
-          <!-- <param name="ip_addr">${ip_addr}</param>
-          <param name="port">${port}</param> -->
       </hardware>
       <joint name="ewellix_lift_top_joint">

Commit message: Added DEXTIVR-221 modifications to avoid merge conflicts

File: ewellix_liftkit_description/urdf/ewellix_lift_700mm.urdf.xacro (robot description, xacro)
@@ -11,4 +11,5 @@
     name="$(arg name)"
     tf_prefix="$(arg tf_prefix)"
+    parent=""
     use_fake_hardware="$(arg use_fake_hardware)"
     com_port="$(arg com_port)"

File: ewellix_liftkit_description/urdf/ewellix_liftkit.ros2_control.xacro (robot description, xacro)
@@ -15,5 +15,5 @@
             <param name="height_limit">${height_limit}</param>
         </hardware>
-        <joint name="${tf_prefix}ewellix_lift_top_joint">
+        <joint name="${tf_prefix}ewellix_lift_lower_to_higher">
           <command_interface name="position"/>
           <state_interface name="position"/>
@@ -28,5 +28,5 @@
             <plugin>mock_components/GenericSystem</plugin>
         </hardware>
-        <joint name="${tf_prefix}ewellix_lift_top_joint">
+        <joint name="${tf_prefix}ewellix_lift_lower_to_higher">
           <command_interface name="position">
             <param name="min">0</param>

File: ewellix_liftkit_description/urdf/ewellix_macro.urdf.xacro (robot description, xacro)
@@ -10,55 +10,125 @@
     height_limit:=0.53
   ">
-    <!-- TODO work on abstracting this xacro to work for both 500 and 700mm lifts -->
+    <!-- TODO figure out how to retract the top link entirely without it colliding through the base. Consider splitting the top into two pieces with a mimic joint (Will do -Mike)-->
+    <!-- Sure hope this is all works in SI units... -Mike-->
+    <!--BASE-->
     <link name="${tf_prefix}ewellix_lift_base_link">
+      <inertia>
+        <mass value="1.7383784"/>
+        <inertia ixx="5.7788770e-03" ixy="0" ixz="0" iyy="7.0031715e-03" iyz="0" izz="1.2717018e-02"/>
+      </inertia>
       <visual>
-        <origin xyz="0 0 0" rpy="0 0 0"/>
         <geometry>
-          <mesh filename="file://$(find ewellix_liftkit_description)/meshes/visual/ewellix_lift_base_700mm.stl"/>
+          <box size="0.220 0.200 0.015"/>
         </geometry>
-        <material name="grey">
-          <color rgba="0.7 0.7 0.7 1"/>
+        <material name="gray">
+          <color rgba="0.85 0.85 0.85 1"/>
         </material>
       </visual>
-      <!-- TODO is this a good collision?-->
       <collision>
-        <origin xyz="-0.005 0 0.00235" rpy="0 0 0"/>
         <geometry>
-          <mesh filename="file://$(find ewellix_liftkit_description)/meshes/visual/ewellix_lift_base_700mm.stl"/>
+          <box size="0.220 0.200 0.015"/>
         </geometry>
       </collision>
     </link>
-    <!-- Lift top link -->
-    <link name="${tf_prefix}ewellix_lift_top_link">
+    <!--LOWER-->
+    <link name="${tf_prefix}ewellix_lift_lower_link">
+      <inertia>
+        <mass value="1.9521070e+01"/>
+        <inertia ixx="0.46604111" ixy="0" ixz="0" iyy="0.46480515" iyz="-0.002668667" izz="0.1561"/>
+      </inertia>
       <visual>
-        <origin xyz="0 0 0" rpy="0 0 0"/>
         <geometry>
-          <mesh filename="file://$(find ewellix_liftkit_description)/meshes/visual/ewellix_lift_top_700mm.stl"/>
+          <mesh filename= "file://$(find ewellix_liftkit_description)/meshes/lift_low.dae"/>
         </geometry>
-        <material name="grey">
-          <color rgba="0.7 0.7 0.7 1"/>
-        </material>
       </visual>
-      <!-- TODO figure out how to retract the top link entirely without it colliding through the base. Consider splitting the top into two pieces with a mimic joint-->
       <collision>
-        <origin xyz="-0.005 0 0.00235" rpy="0 0 0"/>
         <geometry>
-          <mesh filename="file://$(find ewellix_liftkit_description)/meshes/visual/ewellix_lift_top_700mm.stl"/>
+          <box size="0.163 0.163 0.480"/>
         </geometry>
       </collision>
     </link>
-    <!-- Lift base link joint -->
-    <joint name="${tf_prefix}ewellix_lift_base_joint" type="fixed">
-      <parent link="${parent}"/>
-      <child link="${tf_prefix}ewellix_lift_base_link" />
-      <origin xyz="-0.1115 0.0 0.0565" rpy="0 0 3.14159"/>
+    <!--BASE TO LOWER (FIXED)-->
+    <joint name="${tf_prefix}base_to_lower" type="fixed">
+      <parent link="${tf_prefix}ewellix_lift_base_link"/>
+      <child link="${tf_prefix}ewellix_lift_lower_link"/>
+      <origin xyz="0 0 0.2475" rpy="0 0 0"/>
     </joint>
-    <!-- Lift top link joint -->
-    <joint name="${tf_prefix}ewellix_lift_top_joint" type="prismatic">
-      <parent link="${tf_prefix}ewellix_lift_base_link"/>
-      <child link="${tf_prefix}ewellix_lift_top_link" />
-      <origin xyz="0 0 0.730" rpy="0 0 0" />
-      <limit effort="1000" lower="0.0" upper="0.7" velocity="0.088"/>
-      <axis xyz="0 0 1" />
+    <!--MIDDLE-->
+    <link name="${tf_prefix}ewellix_lift_middle_link">
+      <inertia>
+        <mass value="1.5593303e+01"/>
+        <inertia ixx="0.34930648" ixy="0" ixz="0" iyy="0.34930648" iyz="0" izz="0.095393471"/>
+      </inertia>
+      <visual>
+        <geometry>
+          <mesh filename= "file://$(find ewellix_liftkit_description)/meshes/lift_mid.dae"/>
+        </geometry>
+      </visual>
+      <collision>
+        <geometry>
+          <box size="0.146 0.146 0.483"/>
+        </geometry>
+      </collision>
+    </link>
+    <!--HIGHER-->
+    <link name="${tf_prefix}ewellix_lift_higher_link">
+      <inertia>
+        <mass value="1.5166778e+01"/>
+        <inertia ixx="0.35552099" ixy="9.6314989e-6" ixz="2.284786e-5" iyy="0.35552876" iyz="5.4910201e-5" izz="0.069925583"/>
+      </inertia>
+      <visual>
+        <geometry>
+          <mesh filename= "file://$(find ewellix_liftkit_description)/meshes/lift_high.dae"/>
+        </geometry>
+      </visual>
+      <collision>
+        <geometry>
+          <box size="0.129 0.129 0.488"/>
+        </geometry>
+      </collision>
+    </link>
+    <!--LOWER TO HIGHER (PRIS)-->
+    <joint name="${tf_prefix}ewellix_lift_lower_to_higher" type="prismatic">
+      <parent link="${tf_prefix}ewellix_lift_lower_link"/>
+      <child link="${tf_prefix}ewellix_lift_higher_link"/>
+      <origin xyz="0 0 0.0454" rpy="0 0 0"/>
+      <axis xyz="0 0 1"/>
+      <limit lower="0" upper="0.7" effort="1000" velocity="1"/>
+    </joint>
+    <!--MIDDLE MIMIC HIGHER (PRIS MIMIC)-->
+    <joint name="${tf_prefix}ewellix_lift_middle_mimic_higher" type="prismatic">
+      <parent link="${tf_prefix}ewellix_lift_higher_link"/>
+      <child link="${tf_prefix}ewellix_lift_middle_link"/>
+      <origin xyz="0 0 -0.0222" rpy="0 0 0"/>
+      <axis xyz="0 0 -1"/>
+      <limit lower="0" upper="0.351" effort="1000" velocity="1"/>
+      <mimic joint="ewellix_lift_lower_to_higher" multiplier="0.5" offset="0"/>
+    </joint>
+    <!--TOP-->
+    <link name="${tf_prefix}ewellix_lift_top_link">
+      <inertia>
+        <mass value="4.9139525"/>
+        <inertia ixx="0.02015548" ixy="-2.281101e-5" ixz="0" iyy="0.01664141" iyz="0" izz="0.03661307"/>
+      </inertia>
+      <visual>
+        <geometry>
+          <box size="0.200 0.220 0.015"/>
+        </geometry>
+        <material name="gray">
+          <color rgba="0.85 0.85 0.85 1"/>
+        </material>
+      </visual>
+      <collision>
+        <geometry>
+          <box size="0.200 0.220 0.015"/>
+        </geometry>
+      </collision>
+    </link>
+    <!--HIGHER TO TOP (FIXED)-->
+    <joint name="${tf_prefix}ewellix_lift_higher_to_top" type="fixed">
+      <parent link="${tf_prefix}ewellix_lift_higher_link"/>
+      <child link="${tf_prefix}ewellix_lift_top_link"/>
+      <origin xyz="0 0 0.2515" rpy="0 0 0"/>
     </joint>
     <xacro:include filename="$(find ewellix_liftkit_description)/urdf/ewellix_liftkit.ros2_control.xacro" />

Commit message: Added x_offset param. Added another xacro so there's two liftkits.

File: ewellix_liftkit_description/urdf/ewellix_lift_700mm.urdf.xacro (robot description, xacro)
@@ -9,4 +9,5 @@
   <xacro:arg name="use_fake_hardware" default="false" />
   <xacro:arg name="com_port" default="/dev/ttyUSB0" />
+  <xacro:arg name="x_offset" default="0.5" />
   <link name="world"/>
   <xacro:include filename="$(find ewellix_liftkit_description)/urdf/ewellix_lift.xacro"/>
@@ -23,3 +24,14 @@
     <origin xyz="0 0 0" rpy="0 0 0"/>
   </xacro:ewellix_lift>
+  <xacro:ewellix_lift
+    name="$(arg name)_2"
+    tf_prefix="2_"
+    parent="world"
+    height_limit="$(arg height_limit)"
+    omit_plates="false"
+    use_fake_hardware="$(arg use_fake_hardware)"
+    com_port="$(arg com_port)"
+  >
+    <origin xyz="$(arg x_offset) 0 0" rpy="0 0 0"/>
+  </xacro:ewellix_lift>
 </robot>
