Commit message: Renamed ewellix_lift_700mm.urdf.xacro to ewellix_lift.urdf.xacro. Generalized. Can be used for both 500 and 700mm stroke.

File: ewellix_liftkit_description/urdf/ewellix_lift.urdf.xacro (robot description, xacro)
@@ -24,14 +24,3 @@
     <origin xyz="0 0 0" rpy="0 0 0"/>
   </xacro:ewellix_lift>
-  <!-- <xacro:ewellix_lift
-    name="$(arg name)_2"
-    tf_prefix="2_"
-    parent="world"
-    height_limit="$(arg height_limit)"
-    omit_plates="false"
-    use_fake_hardware="$(arg use_fake_hardware)"
-    com_port="$(arg com_port)"
-  >
-    <origin xyz="$(arg x_offset) 0 0" rpy="0 0 0"/>
-  </xacro:ewellix_lift>  -->
 </robot>

Commit message: adding ability to pass in a calibration file

File: ewellix_liftkit_description/urdf/ewellix_lift.urdf.xacro (robot description, xacro)
@@ -11,7 +11,9 @@
   <xacro:arg name="is_700" default="true" />
   <xacro:arg name="is_500" default="false" />
+  <xacro:arg name="hw_calibration_file" default="$(find ewellix_liftkit_description)/config/default_config.yaml"/>
   <link name="world"/>
   <xacro:include filename="$(find ewellix_liftkit_description)/urdf/ewellix_lift.xacro"/>
   <xacro:include filename="$(find ewellix_liftkit_description)/urdf/properties.xacro"/>
+  <xacro:property name="hw_calibration_file" value="$(arg hw_calibration_file)"/>
   <xacro:ewellix_lift
     name="$(arg name)"
@@ -24,4 +26,5 @@
     use_fake_hardware="$(arg use_fake_hardware)"
     com_port="$(arg com_port)"
+    hw_calibration="${xacro.load_yaml(hw_calibration_file)}"
   >
     <origin xyz="0 0 0" rpy="0 0 0"/>

File: ewellix_liftkit_description/urdf/ewellix_lift.xacro (robot description, xacro)
@@ -6,4 +6,5 @@
     parent:=world
     height_limit:=0.7
+    hw_calibration:=${dict(meters_to_ticks=3222.65,ticks_offset=20)}
     omit_plates:=false
     is_700:=true
@@ -275,4 +276,5 @@
       com_port="${com_port}"
       height_limit="${height_limit}"
+      hw_calibration="${hw_calibration}"
     />
   </xacro:macro>

File: ewellix_liftkit_description/urdf/ewellix_liftkit.ros2_control.xacro (robot description, xacro)
@@ -6,5 +6,6 @@
     use_fake_hardware:=false
     com_port:=/dev/ttyUSB0
-    height_limit:=0.7">
+    height_limit:=0.7
+    hw_calibration:=${dict(meters_to_ticks=3222.65,ticks_offset=20)}">
     <xacro:unless value="${use_fake_hardware}">
       <ros2_control name="${name}" type="actuator">
@@ -14,4 +15,6 @@
             <param name="com_port">${com_port}</param>
             <param name="height_limit">${height_limit}</param>
+            <param name="meters_to_ticks">${hw_calibration['meters_to_ticks']}</param>
+            <param name="ticks_offset">${hw_calibration['ticks_offset']}</param>
         </hardware>
         <joint name="${tf_prefix}ewellix_lift_lower_to_higher">

Commit message: Added necessary Gazebo things to the repo to launch Gazebo sim.

File: ewellix_liftkit_description/urdf/ewellix_lift.urdf.xacro (robot description, xacro)
@@ -11,4 +11,5 @@
   <xacro:arg name="is_700" default="true" />
   <xacro:arg name="is_500" default="false" />
+   <xacro:arg name="use_gazebo" default="false" />
   <link name="world"/>
   <xacro:include filename="$(find ewellix_liftkit_description)/urdf/ewellix_lift.xacro"/>
@@ -24,4 +25,5 @@
     use_fake_hardware="$(arg use_fake_hardware)"
     com_port="$(arg com_port)"
+    use_gazebo="$(arg use_gazebo)"
   >
     <origin xyz="0 0 0" rpy="0 0 0"/>

File: ewellix_liftkit_description/urdf/ewellix_lift.xacro (robot description, xacro)
@@ -11,4 +11,5 @@
     use_fake_hardware:=false
     com_port:=/dev/ttyUSB0
+    use_gazebo:=false
     *origin
   ">
@@ -32,5 +33,5 @@
       <xacro:property name="lower_mass_value" value="19.521070"/>
       <xacro:property name="lower_box_size" value="0.163 0.163 0.575"/>
-      <xacro:property name="lower_mesh_filename" value="package://ewellix_liftkit_description/meshes/visual/lift_low_700mm.dae"/>
+      <xacro:property name="lower_mesh_filename" value="file://$(find ewellix_liftkit_description)/meshes/visual/lift_low_700mm.dae"/>
       <xacro:property name="lift_lower_link_ixx" value="0.46604111" scope="parent"/>
       <xacro:property name="lift_lower_link_ixy" value="0.0" scope="parent"/>
@@ -42,5 +43,5 @@
       <xacro:property name="middle_mass_value" value="15.593303"/>
       <xacro:property name="middle_box_size" value="0.146 0.146 0.483"/>
-      <xacro:property name="middle_mesh_filename" value="package://ewellix_liftkit_description/meshes/visual/lift_mid_700mm.dae"/>
+      <xacro:property name="middle_mesh_filename" value="file://$(find ewellix_liftkit_description)/meshes/visual/lift_mid_700mm.dae"/>
       <xacro:property name="lift_middle_link_ixx" value="0.34930648" scope="parent"/>
       <xacro:property name="lift_middle_link_ixy" value="0.0" scope="parent"/>
@@ -50,8 +51,8 @@
       <xacro:property name="lift_middle_link_izz" value="0.095393471" scope="parent"/>
       <xacro:property name="middle_to_higher_origin_z" value="-0.03397"/>
-      <xacro:property name="middle_upper_limit" value="0.351"/>
+      <xacro:property name="middle_upper_limit" value="0.35"/>
       <xacro:property name="higher_mass_value" value="15.166778"/>
       <xacro:property name="higher_box_size" value="0.129 0.129 0.488"/>
-      <xacro:property name="higher_mesh_filename" value="package://ewellix_liftkit_description/meshes/visual/lift_high_700mm.dae"/>
+      <xacro:property name="higher_mesh_filename" value="file://$(find ewellix_liftkit_description)/meshes/visual/lift_high_700mm.dae"/>
       <xacro:property name="lift_higher_link_ixx" value="0.35552099" scope="parent"/>
       <xacro:property name="lift_higher_link_ixy" value="0.000009631" scope="parent"/>
@@ -60,5 +61,5 @@
       <xacro:property name="lift_higher_link_iyz" value="0.000054910" scope="parent"/>
       <xacro:property name="lift_higher_link_izz" value="0.069925583" scope="parent"/>
-      <xacro:property name="higher_to_top_origin_z" value="0.2515"/>
+      <!-- <xacro:property name="higher_to_top_origin_z" value="0.2515"/>
       <xacro:property name="top_mass_value" value="4.9139525"/>
       <xacro:property name="top_box_size" value="0.200 0.220 0.015"/>
@@ -69,5 +70,5 @@
       <xacro:property name="lift_top_link_iyz" value="0.0" scope="parent"/>
       <xacro:property name="lift_top_link_izz" value="0.03661307" scope="parent"/>
-      <xacro:property name="lift_tip_joint_origin_z" value="0.244"/>
+      <xacro:property name="lift_tip_joint_origin_z" value="0.244"/> -->
     </xacro:if>
     <!--For 500 mm stroke-->
@@ -86,7 +87,8 @@
       <xacro:property name="lift_base_link_izz" value="0.012717018" scope="parent"/>
       <xacro:property name="base_to_lower_origin_z" value="0.2457"/>
+      <!-- <xacro:property name="base_to_lower_origin_z" value="0.015"/> -->
       <xacro:property name="lower_mass_value" value="6.746306"/>
       <xacro:property name="lower_box_size" value="0.163 0.163 0.4764"/>
-      <xacro:property name="lower_mesh_filename" value="package://ewellix_liftkit_description/meshes/visual/lift_low_500mm.stl"/>
+      <xacro:property name="lower_mesh_filename" value="file://$(find ewellix_liftkit_description)/meshes/visual/lift_low_500mm.stl"/>
       <xacro:property name="lift_lower_link_ixx" value="0.1579129" scope="parent"/>
       <xacro:property name="lift_lower_link_ixy" value="0" scope="parent"/>
@@ -98,5 +100,5 @@
       <xacro:property name="middle_mass_value" value="5.411604"/>
       <xacro:property name="middle_box_size" value="0.146 0.146 0.4794"/>
-      <xacro:property name="middle_mesh_filename" value="package://ewellix_liftkit_description/meshes/visual/lift_mid_500mm.stl"/>
+      <xacro:property name="middle_mesh_filename" value="file://$(find ewellix_liftkit_description)/meshes/visual/lift_mid_500mm.stl"/>
       <xacro:property name="lift_middle_link_ixx" value="0.11963018" scope="parent"/>
       <xacro:property name="lift_middle_link_ixy" value="0" scope="parent"/>
@@ -109,5 +111,5 @@
       <xacro:property name="higher_mass_value" value="5.324879"/>
       <xacro:property name="higher_box_size" value="0.129 0.129 0.490"/>
-      <xacro:property name="higher_mesh_filename" value="package://ewellix_liftkit_description/meshes/visual/lift_high_500mm.stl"/>
+      <xacro:property name="higher_mesh_filename" value="file://$(find ewellix_liftkit_description)/meshes/visual/lift_high_500mm.stl"/>
       <xacro:property name="lift_higher_link_ixx" value="0.12572077" scope="parent"/>
       <xacro:property name="lift_higher_link_ixy" value="0" scope="parent"/>
@@ -116,6 +118,6 @@
       <xacro:property name="lift_higher_link_iyz" value="0" scope="parent"/>
       <xacro:property name="lift_higher_link_izz" value="0.024552208" scope="parent"/>
-      <xacro:property name="higher_to_top_origin_z" value="0.2525"/>
-      <xacro:property name="top_mass_value" value="1.718423"/>
+      <!-- <xacro:property name="higher_to_top_origin_z" value="0.2525"/> -->
+      <!-- <xacro:property name="top_mass_value" value="1.718423"/>
       <xacro:property name="top_box_size" value="0.200 0.220 0.015"/>
       <xacro:property name="lift_top_link_ixx" value="0.0058195514" scope="parent"/>
@@ -125,5 +127,5 @@
       <xacro:property name="lift_top_link_iyz" value="0.0" scope="parent"/>
       <xacro:property name="lift_top_link_izz" value="0.012803695" scope="parent"/>
-      <xacro:property name="lift_tip_joint_origin_z" value="0.245"/>
+      <xacro:property name="lift_tip_joint_origin_z" value="0.245"/> -->
     </xacro:if>
   <xacro:unless value="${not omit_plates}">
@@ -138,8 +140,8 @@
     <xacro:if value="${not omit_plates}">
       <link name="${tf_prefix}ewellix_lift_base_link">
-        <inertia>
+        <inertial>
           <mass value="${base_mass_value}"/>
           <inertia ixx="${lift_base_link_ixx}" ixy="${lift_base_link_ixy}" ixz="${lift_base_link_ixz}" iyy="${lift_base_link_iyy}" iyz="${lift_base_link_iyz}" izz="${lift_base_link_izz}"/>
-        </inertia>
+        </inertial>
         <visual>
           <geometry>
@@ -157,11 +159,12 @@
     <!--LOWER-->
     <link name="${tf_prefix}ewellix_lift_lower_link">
-      <inertia>
+      <inertial>
         <mass value="${lower_mass_value}"/>
         <inertia ixx="${lift_lower_link_ixx}" ixy="${lift_lower_link_ixy}" ixz="${lift_lower_link_ixz}" iyy="${lift_lower_link_iyy}" iyz="${lift_lower_link_iyz}" izz="${lift_lower_link_izz}"/>
-      </inertia>
+      </inertial>
       <visual>
         <geometry>
-          <mesh filename= "${lower_mesh_filename}"/>
+          <!-- <mesh filename= "${lower_mesh_filename}"/> -->
+          <box size="${lower_box_size}"/>
         </geometry>
         <material name="gray"/>
@@ -183,11 +186,12 @@
     <!--MIDDLE-->
     <link name="${tf_prefix}ewellix_lift_middle_link">
-      <inertia>
+      <inertial>
         <mass value="${middle_mass_value}"/>
         <inertia ixx="${lift_middle_link_ixx}" ixy="${lift_middle_link_ixy}" ixz="${lift_middle_link_ixz}" iyy="${lift_middle_link_iyy}" iyz="${lift_middle_link_iyz}" izz="${lift_middle_link_izz}"/>
-      </inertia>
+      </inertial>
       <visual>
         <geometry>
-          <mesh filename= "${middle_mesh_filename}"/>
+          <!-- <mesh filename= "${middle_mesh_filename}"/> -->
+          <box size="${middle_box_size}"/>
         </geometry>
         <material name="gray"/>
@@ -201,11 +205,12 @@
     <!--HIGHER-->
     <link name="${tf_prefix}ewellix_lift_higher_link">
-      <inertia>
+      <inertial>
         <mass value="${higher_mass_value}"/>
         <inertia ixx="${lift_higher_link_ixx}" ixy="${lift_higher_link_ixy}" ixz="${lift_higher_link_ixz}" iyy="${lift_higher_link_iyy}" iyz="${lift_higher_link_iyz}" izz="${lift_higher_link_izz}"/>
-      </inertia>
+      </inertial>
       <visual>
         <geometry>
-          <mesh filename= "${higher_mesh_filename}"/>
+          <!-- <mesh filename= "${higher_mesh_filename}"/> -->
+          <box size="${higher_box_size}"/>
         </geometry>
         <material name="gray"/>
@@ -234,38 +239,4 @@
       <mimic joint="${tf_prefix}ewellix_lift_lower_to_higher" multiplier="0.5" offset="0"/>
     </joint>
-    <!--TOP (omit_plates=false)-->
-    <xacro:if value="${not omit_plates}">
-      <link name="${tf_prefix}ewellix_lift_top_link">
-        <inertia>
-          <mass value="${top_mass_value}"/>
-          <inertia ixx="${lift_top_link_ixx}" ixy="${lift_top_link_ixy}" ixz="${lift_top_link_ixz}" iyy="${lift_top_link_iyy}" iyz="${lift_top_link_iyz}" izz="${lift_top_link_izz}"/>
-        </inertia>
-        <visual>
-          <geometry>
-            <box size="${top_box_size}"/>
-          </geometry>
-          <material name="gray"/>
-        </visual>
-        <collision>
-          <geometry>
-            <box size="${top_box_size}"/>
-          </geometry>
-        </collision>
-      </link>
-    </xacro:if>
-    <!--HIGHER TO TOP (FIXED, omit_plates=false)-->
-    <xacro:if value="${not omit_plates}">
-      <joint name="${tf_prefix}higher_to_top" type="fixed">
-        <parent link="${tf_prefix}ewellix_lift_higher_link"/>
-        <child link="${tf_prefix}ewellix_lift_top_link"/>
-        <origin xyz="0 0 ${higher_to_top_origin_z}" rpy="0 0 0"/>
-      </joint>
-    </xacro:if>
-    <link name="${tf_prefix}ewellix_lift_tip_link"/>
-    <joint name="${tf_prefix}ewellix_lift_tip_joint" type="fixed">
-      <parent link="${tf_prefix}ewellix_lift_higher_link"/>
-      <child link="${tf_prefix}ewellix_lift_tip_link"/>
-      <origin xyz="0 0 ${lift_tip_joint_origin_z}" rpy="0 0 0"/>
-    </joint>
     <xacro:include filename="$(find ewellix_liftkit_description)/urdf/ewellix_liftkit.ros2_control.xacro" />
     <xacro:ewellix_liftkit_ros2_control
@@ -275,4 +246,5 @@
       com_port="${com_port}"
       height_limit="${height_limit}"
+      use_gazebo="${use_gazebo}"
     />
   </xacro:macro>

File: ewellix_liftkit_description/urdf/ewellix_liftkit.ros2_control.xacro (robot description, xacro)
@@ -6,5 +6,6 @@
     use_fake_hardware:=false
     com_port:=/dev/ttyUSB0
-    height_limit:=0.7">
+    height_limit:=0.7
+    use_gazebo:=false">
     <xacro:unless value="${use_fake_hardware}">
       <ros2_control name="${name}" type="actuator">
@@ -43,4 +44,42 @@
       </ros2_control>
     </xacro:if>
+    <!-- FOR LAUNCHING GAZEBO - Simplified LINKAGE SYSTEM -->
+    <xacro:if value="${use_gazebo}">
+      <ros2_control name="${name}" type="system">
+          <hardware>
+              <plugin>ign_ros2_control/IgnitionSystem</plugin>
+          </hardware>
+          <joint name="${tf_prefix}ewellix_lift_lower_to_higher">
+            <command_interface name="position"/>
+            <state_interface name="position">
+              <param name="initial_value">${height_limit}</param>
+            </state_interface>
+            <state_interface name="velocity"/>
+            <state_interface name="effort"/>
+          </joint>
+          <joint name="${tf_prefix}middle_mimic_higher">
+          <command_interface name="position">
+            <state_interface name="position">
+              <param name="initial_value">${middle_upper_limit}</param>
+            </state_interface>
+            </command_interface>
+            <param name="mimic">${tf_prefix}ewellix_lift_lower_to_higher</param>
+            <param name="multiplier">0.5</param>
+          </joint>
+      </ros2_control>
+      <gazebo>
+        <plugin filename="libign_ros2_control-system.so" name="ign_ros2_control::IgnitionROS2ControlPlugin">
+          <parameters>$(find ewellix_liftkit_deploy)/config/liftkit_controllers.yaml</parameters>
+        </plugin>
+      </gazebo>
+      <gazebo>
+        <plugin filename="libignition-gazebo-pose-publisher-system.so" name="ignition::gazebo::systems::PosePublisher">
+          <publish_link_pose>true</publish_link_pose>
+          <publish_nested_model_pose>true</publish_nested_model_pose>
+          <use_pose_vector_msg>true</use_pose_vector_msg>
+          <update_frequency>50</update_frequency>
+        </plugin>
+      </gazebo>
+    </xacro:if>
   </xacro:macro>
 </robot>
