Commit message: Got ROS2 control working with Elmo controllers and Ewellix actuator, needs some tuning

File: ewellix_liftkit_description/urdf/ewellix_lift.urdf.xacro (robot description, xacro)
@@ -1,21 +1,26 @@
 <?xml version="1.0"?>
-<robot xmlns:xacro="http://wiki.ros.org/xacro" name="$(arg name)">
-  <!-- robot name parameter -->
+<robot xmlns:xacro="http://wiki.ros.org/xacro" name="ewellix_liftkit">
   <xacro:arg name="name" default="ewellix_liftkit"/>
   <xacro:arg name="tf_prefix" default="" />
-  <xacro:arg name="parent" default="" />
+  <xacro:arg name="parent" default="world" />
   <xacro:arg name="height_limit" default="0.7" />
+  <xacro:arg name="initial_value" default="0.0" />
   <xacro:arg name="calibration_direction" default="none" />
   <xacro:arg name="omit_plates" default="false" />
   <xacro:arg name="use_fake_hardware" default="false" />
-  <xacro:arg name="com_port" default="/dev/ttyUSB0" />
+  <xacro:arg name="com_port_top" default="/dev/ttyACM0" />
+  <xacro:arg name="com_port_bottom" default="/dev/ttyACM1" />
   <xacro:arg name="is_700" default="true" />
   <xacro:arg name="is_500" default="false" />
-  <xacro:arg name="hw_calibration_file" default="$(find ewellix_liftkit_description)/config/default_config.yaml"/>
   <xacro:arg name="use_gazebo" default="false" />
+  <xacro:arg name="max_ticks_mot_1" default="872" />
+  <xacro:arg name="max_ticks_mot_2" default="871" />
+  <xacro:arg name="min_height_m" default="0.048" />
+  <xacro:arg name="max_height_m" default="0.587" />
   <link name="world"/>
+  <!-- Include macro files -->
   <xacro:include filename="$(find ewellix_liftkit_description)/urdf/ewellix_lift.xacro"/>
   <xacro:include filename="$(find ewellix_liftkit_description)/urdf/properties.xacro"/>
-  <xacro:property name="hw_calibration_file" value="$(arg hw_calibration_file)"/>
+  <!-- Call the ewellix_lift macro -->
   <xacro:ewellix_lift
     name="$(arg name)"
@@ -23,12 +28,18 @@
     is_500="$(arg is_500)"
     tf_prefix="$(arg tf_prefix)"
-    parent="world"
+    parent="$(arg parent)"
     height_limit="$(arg height_limit)"
+    initial_value="$(arg initial_value)"
     calibration_direction="$(arg calibration_direction)"
-    omit_plates="false"
+    max_ticks_mot_1="$(arg max_ticks_mot_1)"
+    max_ticks_mot_2="$(arg max_ticks_mot_2)"
+    min_height_m="$(arg min_height_m)"
+    max_height_m="$(arg max_height_m)"
+    omit_plates="$(arg omit_plates)"
     use_fake_hardware="$(arg use_fake_hardware)"
-    com_port="$(arg com_port)"
-    hw_calibration="${xacro.load_yaml(hw_calibration_file)}"
+    com_port_top="$(arg com_port_top)"
+    com_port_bottom="$(arg com_port_bottom)"
     use_gazebo="$(arg use_gazebo)"
+    generate_ros2_control_tag="true"
   >
     <origin xyz="0 0 0" rpy="0 0 0"/>

File: ewellix_liftkit_description/urdf/ewellix_lift.xacro (robot description, xacro)
@@ -8,12 +8,16 @@
     initial_value:=0.0
     calibration_direction:=none
-    hw_calibration:=${dict(min_ticks_mot_1=10,min_ticks_mot_2=10,max_ticks_mot_1=800,max_ticks_mot_2=860,min_height_m=0.0,max_height_m=0.7)}
+    max_ticks_mot_1:=800
+    max_ticks_mot_2:=860
+    min_height_m:=0.0
+    max_height_m:=0.7
     omit_plates:=false
     is_700:=true
     is_500:=false
     use_fake_hardware:=false
-    com_port:=/dev/ttyUSB0
+    com_port_top:=/dev/ttyACM0
+    com_port_bottom:=/dev/ttyACM1
     use_gazebo:=false
-    generate_ros2_control_tag=true
+    generate_ros2_control_tag:=true
     *origin
   ">
@@ -132,5 +136,5 @@
       <xacro:property name="lift_tip_joint_origin_z" value="0.245"/>
     </xacro:if>
-  <xacro:unless value="${not omit_plates}">
+    <xacro:unless value="${not omit_plates}">
       <xacro:property name="lift_base_link_name" value="${tf_prefix}ewellix_lift_lower_link"/>
     </xacro:unless>
@@ -168,5 +172,5 @@
       <visual>
         <geometry>
-          <mesh filename= "${lower_mesh_filename}"/>
+          <mesh filename="${lower_mesh_filename}"/>
         </geometry>
         <material name="gray"/>
@@ -194,5 +198,5 @@
       <visual>
         <geometry>
-          <mesh filename= "${middle_mesh_filename}"/>
+          <mesh filename="${middle_mesh_filename}"/>
         </geometry>
         <material name="gray"/>
@@ -212,5 +216,5 @@
       <visual>
         <geometry>
-          <mesh filename= "${higher_mesh_filename}"/>
+          <mesh filename="${higher_mesh_filename}"/>
         </geometry>
         <material name="gray"/>
@@ -239,11 +243,11 @@
       <mimic joint="${tf_prefix}ewellix_lift_lower_to_higher" multiplier="0.5" offset="0"/>
     </joint>
-     <!--TOP (omit_plates=false)-->
+    <!--TOP (omit_plates=false)-->
     <xacro:if value="${not omit_plates}">
       <link name="${tf_prefix}ewellix_lift_top_link">
-        <inertia>
+        <inertial>
           <mass value="${top_mass_value}"/>
           <inertia ixx="${lift_top_link_ixx}" ixy="${lift_top_link_ixy}" ixz="${lift_top_link_ixz}" iyy="${lift_top_link_iyy}" iyz="${lift_top_link_iyz}" izz="${lift_top_link_izz}"/>
-        </inertia>
+        </inertial>
         <visual>
           <geometry>
@@ -273,4 +277,5 @@
       <origin xyz="0 0 ${lift_tip_joint_origin_z}" rpy="0 0 0"/>
     </joint>
+    <!-- ROS2 Control block -->
     <xacro:if value="${generate_ros2_control_tag}">
       <xacro:include filename="$(find ewellix_liftkit_description)/urdf/ewellix_liftkit.ros2_control.xacro" />
@@ -280,10 +285,22 @@
         use_gazebo="${use_gazebo}"
         tf_prefix="${tf_prefix}"
-        com_port="${com_port}"
+        com_port_top="${com_port_top}"
+        com_port_bottom="${com_port_bottom}"
         height_limit="${height_limit}"
         initial_value="${initial_value}"
         calibration_direction="${calibration_direction}"
-        hw_calibration="${hw_calibration}"
-    />
+        max_ticks_mot_1="${max_ticks_mot_1}"
+        max_ticks_mot_2="${max_ticks_mot_2}"
+        min_height_m="${min_height_m}"
+        max_height_m="${max_height_m}"
+        homing_current_a="0.5"
+        stall_velocity_thresh="5"
+        stall_time_ms="400"
+        homing_timeout_ms="15000"
+        poll_ms="20"
+        backoff_counts="500"
+        top_home_direction="1"
+        bottom_home_direction="1"
+      />
     </xacro:if>
   </xacro:macro>

File: ewellix_liftkit_description/urdf/ewellix_liftkit.ros2_control.xacro (robot description, xacro)
@@ -3,76 +3,87 @@
   <xacro:macro name="ewellix_liftkit_ros2_control" params="
     name
-    tf_prefix
+    tf_prefix:=''
     use_fake_hardware:=false
-    com_port:=/dev/ttyUSB0
+    use_gazebo:=false
+    com_port_top:=/dev/ttyACM0
+    com_port_bottom:=/dev/ttyACM1
     height_limit:=0.7
     initial_value:=0.0
     calibration_direction:=none
-    hw_calibration:=${dict(min_ticks_mot_1=10,min_ticks_mot_2=10,max_ticks_mot_1=800,max_ticks_mot_2=860,min_height_m=0.0,max_height_m=0.7)}
-    use_gazebo:=false">
-    <xacro:unless value="${use_fake_hardware}">
-      <ros2_control name="${name}" type="actuator">
+    max_ticks_mot_1:=872
+    max_ticks_mot_2:=871
+    min_height_m:=0.048
+    max_height_m:=0.587
+    homing_current_a:=0.5
+    stall_velocity_thresh:=5
+    stall_time_ms:=400
+    homing_timeout_ms:=15000
+    poll_ms:=20
+    backoff_counts:=500
+    top_home_direction:=1
+    bottom_home_direction:=1">
+    <!-- Single system controlling both motors -->
+    <xacro:if value="${not (use_fake_hardware or use_gazebo)}">
+      <!-- REAL HARDWARE -->
+      <ros2_control name="ewellix_liftkit" type="system">
         <hardware>
-            <plugin>liftkit_hardware_interface/LiftkitHardwareInterface</plugin>
-            <param name="lift_name">liftkit</param>
-            <param name="com_port">${com_port}</param>
-            <param name="height_limit">${height_limit}</param>
-            <param name="calibration_direction">${calibration_direction}</param>
-            <param name="min_ticks_mot_1">${hw_calibration['min_ticks_mot_1']}</param>
-            <param name="min_ticks_mot_2">${hw_calibration['min_ticks_mot_2']}</param>
-            <param name="max_ticks_mot_1">${hw_calibration['max_ticks_mot_1']}</param>
-            <param name="max_ticks_mot_2">${hw_calibration['max_ticks_mot_2']}</param>
-            <param name="min_height_m">${hw_calibration['min_height_m']}</param>
-            <param name="max_height_m">${hw_calibration['max_height_m']}</param>
-        </hardware>
-        <joint name="${tf_prefix}ewellix_lift_lower_to_higher">
-          <command_interface name="position"/>
-          <state_interface name="position"/>
-          <state_interface name="velocity"/>
-          <state_interface name="robot_ready"/>
-        </joint>
-      </ros2_control>
-    </xacro:unless>
-    <xacro:if value="${use_fake_hardware}">
-      <ros2_control name="${name}" type="system">
-        <hardware>
-            <plugin>mock_components/GenericSystem</plugin>
+          <plugin>liftkit_hardware_interface/ElmoLiftkitHardwareInterface</plugin>
+          <param name="com_port_top">${com_port_top}</param>
+          <param name="com_port_bottom">${com_port_bottom}</param>
+          <param name="min_height_m">${min_height_m}</param>
+          <param name="max_height_m">${max_height_m}</param>
+          <param name="max_ticks_mot_1">${max_ticks_mot_1}</param>
+          <param name="max_ticks_mot_2">${max_ticks_mot_2}</param>
+          <param name="homing_current_a">${homing_current_a}</param>
+          <param name="stall_velocity_thresh">${stall_velocity_thresh}</param>
+          <param name="stall_time_ms">${stall_time_ms}</param>
+          <param name="homing_timeout_ms">${homing_timeout_ms}</param>
+          <param name="poll_ms">${poll_ms}</param>
+          <param name="backoff_counts">${backoff_counts}</param>
+          <param name="top_home_direction">${top_home_direction}</param>
+          <param name="bottom_home_direction">${bottom_home_direction}</param>
+          <param name="calibration_direction">${calibration_direction}</param>
+          <param name="height_limit">${height_limit}</param>
         </hardware>
         <joint name="${tf_prefix}ewellix_lift_lower_to_higher">
           <command_interface name="position">
-            <param name="min">0</param>
-            <param name="height_limit">${height_limit}</param>
+            <param name="min">${min_height_m}</param>
+            <param name="max">${max_height_m}</param>
           </command_interface>
-          <state_interface name="position">
-            <param name="initial_value">${initial_value}</param>
-          </state_interface>
+          <state_interface name="position"/>
           <state_interface name="velocity"/>
-          <state_interface name="robot_ready"/>
         </joint>
       </ros2_control>
     </xacro:if>
-    <!-- FOR LAUNCHING GAZEBO -->
-    <xacro:if value="${use_gazebo}">
-      <ros2_control name="${name}" type="system">
-          <hardware>
-              <plugin>ign_ros2_control/IgnitionSystem</plugin>
-          </hardware>
-          <joint name="${tf_prefix}ewellix_lift_lower_to_higher">
-            <command_interface name="position"/>
-            <state_interface name="position">
-              <param name="initial_value">${height_limit}</param>
-            </state_interface>
-            <state_interface name="velocity"/>
-            <state_interface name="effort"/>
-          </joint>
-          <joint name="${tf_prefix}middle_mimic_higher">
+    <!-- FAKE HARDWARE -->
+    <xacro:if value="${use_fake_hardware}">
+      <ros2_control name="ewellix_liftkit" type="system">
+        <hardware>
+          <plugin>liftkit_hardware_interface/ElmoLiftkitHardwareInterface</plugin>
+          <param name="com_port_top">/dev/null</param>
+          <param name="com_port_bottom">/dev/null</param>
+          <param name="min_height_m">${min_height_m}</param>
+          <param name="max_height_m">${max_height_m}</param>
+          <param name="max_ticks_mot_1">${max_ticks_mot_1}</param>
+          <param name="max_ticks_mot_2">${max_ticks_mot_2}</param>
+          <param name="homing_current_a">${homing_current_a}</param>
+          <param name="stall_velocity_thresh">${stall_velocity_thresh}</param>
+          <param name="stall_time_ms">${stall_time_ms}</param>
+          <param name="homing_timeout_ms">${homing_timeout_ms}</param>
+          <param name="poll_ms">${poll_ms}</param>
+          <param name="backoff_counts">${backoff_counts}</param>
+          <param name="top_home_direction">${top_home_direction}</param>
+          <param name="bottom_home_direction">${bottom_home_direction}</param>
+          <param name="calibration_direction">${calibration_direction}</param>
+          <param name="height_limit">${height_limit}</param>
+        </hardware>
+        <joint name="${tf_prefix}ewellix_lift_lower_to_higher">
           <command_interface name="position">
-            <state_interface name="position">
-              <param name="initial_value">${middle_upper_limit}</param>
-            </state_interface>
-            </command_interface>
-            <param name="mimic">${tf_prefix}ewellix_lift_lower_to_higher</param>
-            <param name="multiplier">0.5</param>
-          </joint>
+            <param name="min">${min_height_m}</param>
+            <param name="max">${max_height_m}</param>
+          </command_interface>
+          <state_interface name="position"/>
+          <state_interface name="velocity"/>
+        </joint>
       </ros2_control>
     </xacro:if>
