Commit message: addressed merge comments, placed material properties in properties.xacro and imported for use, removed the 'urdf' from the ewellix_lift macro file name, added argument for max height (to add 500mm lift compatibility) but it doesn't work

File: ewellix_liftkit_description/urdf/ewellix_lift.xacro (robot description, xacro)
@@ -1,16 +1,14 @@
 <?xml version="1.0"?>
 <robot xmlns:xacro="http://www.ros.org/wiki/xacro">
-  <xacro:property name="M_PI" value="3.1415926535897931" />
+  <xacro:include filename="$(find ewellix_liftkit_description)/urdf/properties.xacro"/>
   <xacro:macro name="ewellix_lift" params="
     name
     tf_prefix
+    max_height:=700
     use_fake_hardware:=false
     com_port:=/dev/ttyUSB0
     baudrate:=34800
   ">
-    <!-- TODO work on abstracting this xacro to work for both 500 and 700mm lifts (I'll give it a shot -Mike)-->
-    <!-- TODO is this a good collision? (No, it wasn't, raw meshes in general do not make good collision objects -Mike)-->
-    <!-- TODO figure out how to retract the top link entirely without it colliding through the base. Consider splitting the top into two pieces with a mimic joint (Will do -Mike)-->
-    <!-- Sure hope this is all works in SI units... -Mike-->
+    <!-- TODO work on abstracting this xacro to work for both 500 and 700mm lifts-->
     <!--BASE-->
     <link name="${tf_prefix}ewellix_lift_base_link">
@@ -23,7 +21,5 @@
           <box size="0.220 0.200 0.015"/>
         </geometry>
-        <material name="gray">
-          <color rgba="0.85 0.85 0.85 1"/>
-        </material>
+        <material name="gray"/>
       </visual>
       <collision>
@@ -43,4 +39,5 @@
           <mesh filename= "file://$(find ewellix_liftkit_description)/meshes/visual/lift_low.dae"/>
         </geometry>
+        <material name="gray"/>
       </visual>
       <collision>
@@ -66,4 +63,5 @@
           <mesh filename= "file://$(find ewellix_liftkit_description)/meshes/visual/lift_mid.dae"/>
         </geometry>
+        <material name="gray"/>
       </visual>
       <collision>
@@ -83,4 +81,5 @@
           <mesh filename= "file://$(find ewellix_liftkit_description)/meshes/visual/lift_high.dae"/>
         </geometry>
+        <material name="gray"/>
       </visual>
       <collision>
@@ -96,5 +95,5 @@
       <origin xyz="0 0 0.0454" rpy="0 0 0"/>
       <axis xyz="0 0 1"/>
-      <limit lower="0" upper="0.7" effort="1000" velocity="1"/>
+      <limit lower="0" upper="${max_height / 1000.0}" effort="1000" velocity="1"/>
     </joint>
     <!--MIDDLE MIMIC HIGHER (PRIS MIMIC)-->
@@ -117,7 +116,5 @@
           <box size="0.200 0.220 0.015"/>
         </geometry>
-        <material name="gray">
-          <color rgba="0.85 0.85 0.85 1"/>
-        </material>
+        <material name="gray"/>
       </visual>
       <collision>

File: ewellix_liftkit_description/urdf/ewellix_lift_700mm.urdf.xacro (robot description, xacro)
@@ -7,5 +7,5 @@
   <xacro:arg name="com_port" default="/dev/ttyUSB0" />
   <xacro:arg name="baudrate" default="34800" />
-  <xacro:include filename="$(find ewellix_liftkit_description)/urdf/ewellix_macro.urdf.xacro"/>
+  <xacro:include filename="$(find ewellix_liftkit_description)/urdf/ewellix_lift.xacro"/>
   <xacro:ewellix_lift
     name="$(arg name)"

Commit message: parameter fixes that were needed from merging, added height_limit and removed baudrate

File: ewellix_liftkit_description/urdf/ewellix_lift.xacro (robot description, xacro)
@@ -5,8 +5,8 @@
     name
     tf_prefix
-    max_height:=700
+    parent
+    height_limit:=0.7
     use_fake_hardware:=false
     com_port:=/dev/ttyUSB0
-    baudrate:=34800
   ">
     <!-- TODO work on abstracting this xacro to work for both 500 and 700mm lifts-->
@@ -95,5 +95,5 @@
       <origin xyz="0 0 0.0454" rpy="0 0 0"/>
       <axis xyz="0 0 1"/>
-      <limit lower="0" upper="${max_height / 1000.0}" effort="1000" velocity="1"/>
+      <limit lower="0" upper="${height_limit}" effort="1000" velocity="1"/>
     </joint>
     <!--MIDDLE MIMIC HIGHER (PRIS MIMIC)-->
@@ -136,5 +136,5 @@
       tf_prefix="${tf_prefix}"
       com_port="${com_port}"
-      baudrate="${baudrate}"
+      height_limit="${height_limit}"
     />
   </xacro:macro>

Commit message: Added omit_plates option to ewellix_lift macro, optionally removes upper and lower plates

File: ewellix_liftkit_description/urdf/ewellix_lift.xacro (robot description, xacro)
@@ -7,26 +7,29 @@
     parent
     height_limit:=0.7
+    omit_plates:=false
     use_fake_hardware:=false
     com_port:=/dev/ttyUSB0
   ">
     <!-- TODO work on abstracting this xacro to work for both 500 and 700mm lifts-->
-    <!--BASE-->
-    <link name="${tf_prefix}ewellix_lift_base_link">
-      <inertia>
-        <mass value="1.7383784"/>
-        <inertia ixx="5.7788770e-03" ixy="0" ixz="0" iyy="7.0031715e-03" iyz="0" izz="1.2717018e-02"/>
-      </inertia>
-      <visual>
-        <geometry>
-          <box size="0.220 0.200 0.015"/>
-        </geometry>
-        <material name="gray"/>
-      </visual>
-      <collision>
-        <geometry>
-          <box size="0.220 0.200 0.015"/>
-        </geometry>
-      </collision>
-    </link>
+    <!--BASE (omit_plates=false)-->
+    <xacro:if value="${not omit_plates}">
+      <link name="${tf_prefix}ewellix_lift_base_link">
+        <inertia>
+          <mass value="1.7383784"/>
+          <inertia ixx="5.7788770e-03" ixy="0" ixz="0" iyy="7.0031715e-03" iyz="0" izz="1.2717018e-02"/>
+        </inertia>
+        <visual>
+          <geometry>
+            <box size="0.220 0.200 0.015"/>
+          </geometry>
+          <material name="gray"/>
+        </visual>
+        <collision>
+          <geometry>
+            <box size="0.220 0.200 0.015"/>
+          </geometry>
+        </collision>
+      </link>
+    </xacro:if>
     <!--LOWER-->
     <link name="${tf_prefix}ewellix_lift_lower_link">
@@ -47,10 +50,12 @@
       </collision>
     </link>
-    <!--BASE TO LOWER (FIXED)-->
-    <joint name="base_to_lower" type="fixed">
-      <parent link="${tf_prefix}ewellix_lift_base_link"/>
-      <child link="${tf_prefix}ewellix_lift_lower_link"/>
-      <origin xyz="0 0 0.2475" rpy="0 0 0"/>
-    </joint>
+    <!--BASE TO LOWER (FIXED, omit_plates=false)-->
+    <xacro:if value="${not omit_plates}">
+      <joint name="base_to_lower" type="fixed">
+        <parent link="${tf_prefix}ewellix_lift_base_link"/>
+        <child link="${tf_prefix}ewellix_lift_lower_link"/>
+        <origin xyz="0 0 0.2475" rpy="0 0 0"/>
+      </joint>
+    </xacro:if>
     <!--MIDDLE-->
     <link name="${tf_prefix}ewellix_lift_middle_link">
@@ -107,27 +112,31 @@
     </joint>
     <!--TOP-->
-    <link name="${tf_prefix}ewellix_lift_top_link">
-      <inertia>
-        <mass value="4.9139525"/>
-        <inertia ixx="0.02015548" ixy="-2.281101e-5" ixz="0" iyy="0.01664141" iyz="0" izz="0.03661307"/>
-      </inertia>
-      <visual>
-        <geometry>
-          <box size="0.200 0.220 0.015"/>
-        </geometry>
-        <material name="gray"/>
-      </visual>
-      <collision>
-        <geometry>
-          <box size="0.200 0.220 0.015"/>
-        </geometry>
-      </collision>
-    </link>
+    <xacro:if value="${not omit_plates}">
+      <link name="${tf_prefix}ewellix_lift_top_link">
+        <inertia>
+          <mass value="4.9139525"/>
+          <inertia ixx="0.02015548" ixy="-2.281101e-5" ixz="0" iyy="0.01664141" iyz="0" izz="0.03661307"/>
+        </inertia>
+        <visual>
+          <geometry>
+            <box size="0.200 0.220 0.015"/>
+          </geometry>
+          <material name="gray"/>
+        </visual>
+        <collision>
+          <geometry>
+            <box size="0.200 0.220 0.015"/>
+          </geometry>
+        </collision>
+      </link>
+    </xacro:if>
     <!--HIGHER TO TOP (FIXED)-->
-    <joint name="higher_to_top" type="fixed">
-      <parent link="${tf_prefix}ewellix_lift_higher_link"/>
-      <child link="${tf_prefix}ewellix_lift_top_link"/>
-      <origin xyz="0 0 0.2515" rpy="0 0 0"/>
-    </joint>
+    <xacro:if value="${not omit_plates}">
+      <joint name="higher_to_top" type="fixed">
+        <parent link="${tf_prefix}ewellix_lift_higher_link"/>
+        <child link="${tf_prefix}ewellix_lift_top_link"/>
+        <origin xyz="0 0 0.2515" rpy="0 0 0"/>
+      </joint>
+    </xacro:if>
     <xacro:include filename="$(find ewellix_liftkit_description)/urdf/ewellix_liftkit.ros2_control.xacro" />
     <xacro:ewellix_liftkit_ros2_control

File: ewellix_liftkit_description/urdf/ewellix_lift_700mm.urdf.xacro (robot description, xacro)
@@ -4,7 +4,9 @@
   <xacro:arg name="name" default="ewellix_liftkit"/>
   <xacro:arg name="tf_prefix" default="" />
+  <xacro:arg name="parent" default="" />
+  <xacro:arg name="height_limit" default="0.7" />
+  <xacro:arg name="omit_plates" default="false" />
   <xacro:arg name="use_fake_hardware" default="false" />
   <xacro:arg name="com_port" default="/dev/ttyUSB0" />
-  <xacro:arg name="height_limit" default="0.53" />
   <xacro:include filename="$(find ewellix_liftkit_description)/urdf/ewellix_lift.xacro"/>
   <xacro:ewellix_lift
@@ -12,6 +14,8 @@
     tf_prefix="$(arg tf_prefix)"
     parent=""
+    height_limit="$(arg height_limit)"
+    omit_plates="false"
     use_fake_hardware="$(arg use_fake_hardware)"
     com_port="$(arg com_port)"
-    height_limit="$(arg height_limit)"/>
+    />
 </robot>

Commit message: fixed joint name to match ros2 control and moveit

File: ewellix_liftkit_description/urdf/ewellix_lift.xacro (robot description, xacro)
@@ -96,5 +96,5 @@
     <!-- TODO Limit Upper Height -Mike -->
     <!--LOWER TO HIGHER (PRIS)-->
-    <joint name="lower_to_higher" type="prismatic">
+    <joint name="ewellix_lift_lower_to_higher" type="prismatic">
       <parent link="${tf_prefix}ewellix_lift_lower_link"/>
       <child link="${tf_prefix}ewellix_lift_higher_link"/>
@@ -110,5 +110,5 @@
       <axis xyz="0 0 -1"/>
       <limit lower="0" upper="0.351" effort="1000" velocity="1"/>
-      <mimic joint="lower_to_higher" multiplier="0.5" offset="0"/>
+      <mimic joint="ewellix_lift_lower_to_higher" multiplier="0.5" offset="0"/>
     </joint>
     <!--TOP (omit_plates=false)-->

Commit message: absctracted base joint, exposed parent and origin in lift macro

File: ewellix_liftkit_description/urdf/ewellix_lift.xacro (robot description, xacro)
@@ -4,12 +4,24 @@
   <xacro:macro name="ewellix_lift" params="
     name
-    tf_prefix
-    parent
+    tf_prefix:=''
+    parent:=world
     height_limit:=0.7
     omit_plates:=false
     use_fake_hardware:=false
     com_port:=/dev/ttyUSB0
+    *origin
   ">
     <!-- TODO work on abstracting this xacro to work for both 500 and 700mm lifts-->
+    <xacro:if value="${not omit_plates}">
+      <xacro:property name="lift_base_link_name" value="${tf_prefix}ewellix_lift_base_link"/>
+    </xacro:if>
+    <xacro:unless value="${not omit_plates}">
+      <xacro:property name="lift_base_link_name" value="${tf_prefix}ewellix_lift_lower_link"/>
+    </xacro:unless>
+    <joint name="${tf_prefix}ewellix_lift_base_joint" type="fixed">
+      <parent link="${parent}"/>
+      <child link="${lift_base_link_name}"/>
+      <xacro:insert_block name="origin"/>
+    </joint>
     <!--BASE (omit_plates=false)-->
     <xacro:if value="${not omit_plates}">

File: ewellix_liftkit_description/urdf/ewellix_lift_700mm.urdf.xacro (robot description, xacro)
@@ -13,9 +13,11 @@
     name="$(arg name)"
     tf_prefix="$(arg tf_prefix)"
-    parent=""
+    parent="world"
     height_limit="$(arg height_limit)"
     omit_plates="false"
     use_fake_hardware="$(arg use_fake_hardware)"
     com_port="$(arg com_port)"
-    />
+  >
+    <origin xyz="0 0 0" rpy="0 0 0"/>
+  </xacro:ewellix_lift>
 </robot>

Commit message: added lift tip

File: ewellix_liftkit_description/urdf/ewellix_lift.xacro (robot description, xacro)
@@ -152,4 +152,10 @@
       </joint>
     </xacro:if>
+    <link name="${tf_prefix}ewellix_lift_tip_link"/>
+    <joint name="${tf_prefix}ewellix_lift_tip_joint" type="fixed">
+      <parent link="${tf_prefix}ewellix_lift_higher_link"/>
+      <child link="${tf_prefix}ewellix_lift_tip_link"/>
+      <origin xyz="0 0 0.244" rpy="0 0 0"/>
+    </joint>
     <xacro:include filename="$(find ewellix_liftkit_description)/urdf/ewellix_liftkit.ros2_control.xacro" />
     <xacro:ewellix_liftkit_ros2_control

File: ewellix_liftkit_description/urdf/ewellix_lift_700mm.urdf.xacro (robot description, xacro)
@@ -9,4 +9,5 @@
   <xacro:arg name="use_fake_hardware" default="false" />
   <xacro:arg name="com_port" default="/dev/ttyUSB0" />
+  <link name="world"/>
   <xacro:include filename="$(find ewellix_liftkit_description)/urdf/ewellix_lift.xacro"/>
   <xacro:ewellix_lift

Commit message: file to package ref

File: ewellix_liftkit_description/urdf/ewellix_lift.xacro (robot description, xacro)
@@ -52,5 +52,5 @@
       <visual>
         <geometry>
-          <mesh filename= "file://$(find ewellix_liftkit_description)/meshes/visual/lift_low.dae"/>
+          <mesh filename= "package://ewellix_liftkit_description/meshes/visual/lift_low.dae"/>
         </geometry>
         <material name="gray"/>
@@ -78,5 +78,5 @@
       <visual>
         <geometry>
-          <mesh filename= "file://$(find ewellix_liftkit_description)/meshes/visual/lift_mid.dae"/>
+          <mesh filename= "package://ewellix_liftkit_description/meshes/visual/lift_mid.dae"/>
         </geometry>
         <material name="gray"/>
@@ -96,5 +96,5 @@
       <visual>
         <geometry>
-          <mesh filename= "file://$(find ewellix_liftkit_description)/meshes/visual/lift_high.dae"/>
+          <mesh filename= "package://ewellix_liftkit_description/meshes/visual/lift_high.dae"/>
         </geometry>
         <material name="gray"/>

Commit message: replaced lift_low mesh, increased height from an incorrect 480mm to an accurate 575mm, updated lift macro origins

File: ewellix_liftkit_description/urdf/ewellix_lift.xacro (robot description, xacro)
@@ -58,5 +58,5 @@
       <collision>
         <geometry>
-          <box size="0.163 0.163 0.480"/>
+          <box size="0.163 0.163 0.575"/>
         </geometry>
       </collision>
@@ -67,5 +67,5 @@
         <parent link="${tf_prefix}ewellix_lift_base_link"/>
         <child link="${tf_prefix}ewellix_lift_lower_link"/>
-        <origin xyz="0 0 0.2475" rpy="0 0 0"/>
+        <origin xyz="0 0 0.295" rpy="0 0 0"/>
       </joint>
     </xacro:if>
@@ -111,5 +111,5 @@
       <parent link="${tf_prefix}ewellix_lift_lower_link"/>
       <child link="${tf_prefix}ewellix_lift_higher_link"/>
-      <origin xyz="0 0 0.0454" rpy="0 0 0"/>
+      <origin xyz="0 0 0.0915" rpy="0 0 0"/>
       <axis xyz="0 0 1"/>
       <limit lower="0" upper="${height_limit}" effort="1000" velocity="1"/>
@@ -119,5 +119,5 @@
       <parent link="${tf_prefix}ewellix_lift_higher_link"/>
       <child link="${tf_prefix}ewellix_lift_middle_link"/>
-      <origin xyz="0 0 -0.0222" rpy="0 0 0"/>
+      <origin xyz="0 0 -0.03397" rpy="0 0 0"/>
       <axis xyz="0 0 -1"/>
       <limit lower="0" upper="0.351" effort="1000" velocity="1"/>

Commit message: Added tf_prefix to all joints. For calling multiple liftkits.

File: ewellix_liftkit_description/urdf/ewellix_lift.xacro (robot description, xacro)
@@ -12,7 +12,42 @@
   ">
     <!-- TODO work on abstracting this xacro to work for both 500 and 700mm lifts-->
+    <!-- do not put any special characters such as a colon in a comment in xacros-->
     <xacro:if value="${not omit_plates}">
       <xacro:property name="lift_base_link_name" value="${tf_prefix}ewellix_lift_base_link"/>
     </xacro:if>
+    <!--
+    <xacro:if value="500">
+    <xacro:property name="lift_base_link_ixx" value="0.0" scope="parent"/>
+    <xacro:property name="lift_base_link_ixy" value="0.0" scope="parent"/>
+    <xacro:property name="lift_base_link_ixz" value="0.0" scope="parent"/>
+    <xacro:property name="lift_base_link_iyy" value="0.0" scope="parent"/>
+    <xacro:property name="lift_base_link_iyz" value="0.0" scope="parent"/>
+    <xacro:property name="lift_base_link_izz" value="0.0" scope="parent"/>
+    <xacro:property name="lift_lower_link_ixx" value="0.0" scope="parent"/>
+    <xacro:property name="lift_lower_link_ixy" value="0.0" scope="parent"/>
+    <xacro:property name="lift_lower_link_ixz" value="0.0" scope="parent"/>
+    <xacro:property name="lift_lower_link_iyy" value="0.0" scope="parent"/>
+    <xacro:property name="lift_lower_link_iyz" value="0.0" scope="parent"/>
+    <xacro:property name="lift_lower_link_izz" value="0.0" scope="parent"/>
+    <xacro:property name="lift_middle_link_ixx" value="0.0" scope="parent"/>
+    <xacro:property name="lift_middle_link_ixy" value="0.0" scope="parent"/>
+    <xacro:property name="lift_middle_link_ixz" value="0.0" scope="parent"/>
+    <xacro:property name="lift_middle_link_iyy" value="0.0" scope="parent"/>
+    <xacro:property name="lift_middle_link_iyz" value="0.0" scope="parent"/>
+    <xacro:property name="lift_middle_link_izz" value="0.0" scope="parent"/>
+    <xacro:property name="lift_higher_link_ixx" value="0.0" scope="parent"/>
+    <xacro:property name="lift_higher_link_ixy" value="0.0" scope="parent"/>
+    <xacro:property name="lift_higher_link_ixz" value="0.0" scope="parent"/>
+    <xacro:property name="lift_higher_link_iyy" value="0.0" scope="parent"/>
+    <xacro:property name="lift_higher_link_iyz" value="0.0" scope="parent"/>
+    <xacro:property name="lift_higher_link_izz" value="0.0" scope="parent"/>
+    <xacro:property name="lift_top_link_ixx" value="0.0" scope="parent"/>
+    <xacro:property name="lift_top_link_ixy" value="0.0" scope="parent"/>
+    <xacro:property name="lift_top_link_ixz" value="0.0" scope="parent"/>
+    <xacro:property name="lift_top_link_iyy" value="0.0" scope="parent"/>
+    <xacro:property name="lift_top_link_iyz" value="0.0" scope="parent"/>
+    <xacro:property name="lift_top_link_izz" value="0.0" scope="parent"/>
+    </xacro:if>
+    -->
     <xacro:unless value="${not omit_plates}">
       <xacro:property name="lift_base_link_name" value="${tf_prefix}ewellix_lift_lower_link"/>
@@ -63,5 +98,5 @@
     <!--BASE TO LOWER (FIXED, omit_plates=false)-->
     <xacro:if value="${not omit_plates}">
-      <joint name="base_to_lower" type="fixed">
+      <joint name="${tf_prefix}base_to_lower" type="fixed">
         <parent link="${tf_prefix}ewellix_lift_base_link"/>
         <child link="${tf_prefix}ewellix_lift_lower_link"/>
@@ -107,5 +142,5 @@
     <!-- TODO Limit Upper Height -Mike -->
     <!--LOWER TO HIGHER (PRISMATIC)-->
-    <joint name="ewellix_lift_lower_to_higher" type="prismatic">
+    <joint name="${tf_prefix}ewellix_lift_lower_to_higher" type="prismatic">
       <parent link="${tf_prefix}ewellix_lift_lower_link"/>
       <child link="${tf_prefix}ewellix_lift_higher_link"/>
@@ -115,5 +150,5 @@
     </joint>
     <!--MIDDLE MIMIC HIGHER (PRISMATIC MIMIC)-->
-    <joint name="middle_mimic_higher" type="prismatic">
+    <joint name="${tf_prefix}middle_mimic_higher" type="prismatic">
       <parent link="${tf_prefix}ewellix_lift_higher_link"/>
       <child link="${tf_prefix}ewellix_lift_middle_link"/>
@@ -121,5 +156,5 @@
       <axis xyz="0 0 -1"/>
       <limit lower="0" upper="0.351" effort="1000" velocity="1"/>
-      <mimic joint="ewellix_lift_lower_to_higher" multiplier="0.5" offset="0"/>
+      <mimic joint="${tf_prefix}ewellix_lift_lower_to_higher" multiplier="0.5" offset="0"/>
     </joint>
     <!--TOP (omit_plates=false)-->
@@ -145,5 +180,5 @@
     <!--HIGHER TO TOP (FIXED, omit_plates=false)-->
     <xacro:if value="${not omit_plates}">
-      <joint name="higher_to_top" type="fixed">
+      <joint name="${tf_prefix}higher_to_top" type="fixed">
         <parent link="${tf_prefix}ewellix_lift_higher_link"/>
         <child link="${tf_prefix}ewellix_lift_top_link"/>
