Commit message: Modified such that hard-coded values are now parameters. Now this xacro can be used for both 500 and 700 mm stroke. Abstract tested and successful. Just need to add values for the 500 mm liftkit parameters.

File: ewellix_liftkit_description/urdf/ewellix_lift.xacro (robot description, xacro)
@@ -7,4 +7,5 @@
     height_limit:=0.7
     omit_plates:=false
+    is_700:=true
     use_fake_hardware:=false
     com_port:=/dev/ttyUSB0
@@ -16,6 +17,53 @@
       <xacro:property name="lift_base_link_name" value="${tf_prefix}ewellix_lift_base_link"/>
     </xacro:if>
-    <!--
+    <xacro:if value="${is_700}">
+    <xacro:property name="base_mass_value" value="1.7383784"/>
+    <xacro:property name="base_box_size" value="0.220 0.200 0.015"/>
+    <xacro:property name="lift_base_link_ixx" value="5.7788770e-03" scope="parent"/>
+    <xacro:property name="lift_base_link_ixy" value="0.0" scope="parent"/>
+    <xacro:property name="lift_base_link_ixz" value="0.0" scope="parent"/>
+    <xacro:property name="lift_base_link_iyy" value="7.0031715e-03" scope="parent"/>
+    <xacro:property name="lift_base_link_iyz" value="0.0" scope="parent"/>
+    <xacro:property name="lift_base_link_izz" value="1.2717018e-02" scope="parent"/>
+    <xacro:property name="lower_mass_value" value="1.9521070e+01"/>
+    <xacro:property name="lower_box_size" value="0.163 0.163 0.575"/>
+    <xacro:property name="lower_mesh_filename" value="package://ewellix_liftkit_description/meshes/visual/lift_low.dae"/>
+    <xacro:property name="lift_lower_link_ixx" value="0.46604111" scope="parent"/>
+    <xacro:property name="lift_lower_link_ixy" value="0.0" scope="parent"/>
+    <xacro:property name="lift_lower_link_ixz" value="0.0" scope="parent"/>
+    <xacro:property name="lift_lower_link_iyy" value="0.46480515" scope="parent"/>
+    <xacro:property name="lift_lower_link_iyz" value="-0.002668667" scope="parent"/>
+    <xacro:property name="lift_lower_link_izz" value="0.1561" scope="parent"/>
+    <xacro:property name="middle_mass_value" value="1.5593303e+01"/>
+    <xacro:property name="middle_box_size" value="0.146 0.146 0.483"/>
+    <xacro:property name="middle_mesh_filename" value="package://ewellix_liftkit_description/meshes/visual/lift_mid.dae"/>
+    <xacro:property name="lift_middle_link_ixx" value="0.34930648" scope="parent"/>
+    <xacro:property name="lift_middle_link_ixy" value="0.0" scope="parent"/>
+    <xacro:property name="lift_middle_link_ixz" value="0.0" scope="parent"/>
+    <xacro:property name="lift_middle_link_iyy" value="0.34930648" scope="parent"/>
+    <xacro:property name="lift_middle_link_iyz" value="0.0" scope="parent"/>
+    <xacro:property name="lift_middle_link_izz" value="0.095393471" scope="parent"/>
+    <xacro:property name="higher_mass_value" value="1.5166778e+01"/>
+    <xacro:property name="higher_box_size" value="0.129 0.129 0.488"/>
+    <xacro:property name="higher_mesh_filename" value="package://ewellix_liftkit_description/meshes/visual/lift_high.dae"/>
+    <xacro:property name="lift_higher_link_ixx" value="0.35552099" scope="parent"/>
+    <xacro:property name="lift_higher_link_ixy" value="9.6314989e-6" scope="parent"/>
+    <xacro:property name="lift_higher_link_ixz" value="2.284786e-5" scope="parent"/>
+    <xacro:property name="lift_higher_link_iyy" value="0.35552876" scope="parent"/>
+    <xacro:property name="lift_higher_link_iyz" value="5.4910201e-5" scope="parent"/>
+    <xacro:property name="lift_higher_link_izz" value="0.069925583" scope="parent"/>
+    <xacro:property name="top_mass_value" value="4.9139525"/>
+    <xacro:property name="top_box_size" value="0.200 0.220 0.015"/>
+    <xacro:property name="lift_top_link_ixx" value="0.02015548" scope="parent"/>
+    <xacro:property name="lift_top_link_ixy" value="-2.281101e-5" scope="parent"/>
+    <xacro:property name="lift_top_link_ixz" value="0.0" scope="parent"/>
+    <xacro:property name="lift_top_link_iyy" value="0.01664141" scope="parent"/>
+    <xacro:property name="lift_top_link_iyz" value="0.0" scope="parent"/>
+    <xacro:property name="lift_top_link_izz" value="0.03661307" scope="parent"/>
+    </xacro:if>
+     <!--
     <xacro:if value="500">
+    <xacro:property name="base_mass_value" value="0.0"/>
+    <xacro:property name="base_box_size" value="0.0 0.0 0.0"/>
     <xacro:property name="lift_base_link_ixx" value="0.0" scope="parent"/>
     <xacro:property name="lift_base_link_ixy" value="0.0" scope="parent"/>
@@ -24,4 +72,7 @@
     <xacro:property name="lift_base_link_iyz" value="0.0" scope="parent"/>
     <xacro:property name="lift_base_link_izz" value="0.0" scope="parent"/>
+    <xacro:property name="lower_mass_value" value="0.0"/>
+    <xacro:property name="lower_box_size" value="0.0 0.0 0.0"/>
+    <xacro:property name="lower_mesh_filename" value="..."/>
     <xacro:property name="lift_lower_link_ixx" value="0.0" scope="parent"/>
     <xacro:property name="lift_lower_link_ixy" value="0.0" scope="parent"/>
@@ -30,4 +81,7 @@
     <xacro:property name="lift_lower_link_iyz" value="0.0" scope="parent"/>
     <xacro:property name="lift_lower_link_izz" value="0.0" scope="parent"/>
+    <xacro:property name="middle_mass_value" value="0.0"/>
+    <xacro:property name="middle_box_size" value="0.0 0.0 0.0"/>
+    <xacro:property name="middle_mesh_filename" value="..."/>
     <xacro:property name="lift_middle_link_ixx" value="0.0" scope="parent"/>
     <xacro:property name="lift_middle_link_ixy" value="0.0" scope="parent"/>
@@ -36,4 +90,7 @@
     <xacro:property name="lift_middle_link_iyz" value="0.0" scope="parent"/>
     <xacro:property name="lift_middle_link_izz" value="0.0" scope="parent"/>
+    <xacro:property name="higher_mass_value" value="0.0"/>
+    <xacro:property name="higher_box_size" value="0.0 0.0 0.0"/>
+    <xacro:property name="higher_mesh_filename" value="..."/>
     <xacro:property name="lift_higher_link_ixx" value="0.0" scope="parent"/>
     <xacro:property name="lift_higher_link_ixy" value="0.0" scope="parent"/>
@@ -62,10 +119,10 @@
       <link name="${tf_prefix}ewellix_lift_base_link">
         <inertia>
-          <mass value="1.7383784"/>
-          <inertia ixx="5.7788770e-03" ixy="0" ixz="0" iyy="7.0031715e-03" iyz="0" izz="1.2717018e-02"/>
+          <mass value="${base_mass_value}"/>
+          <inertia ixx="${lift_base_link_ixx}" ixy="${lift_base_link_ixy}" ixz="${lift_base_link_ixz}" iyy="${lift_base_link_iyy}" iyz="${lift_base_link_iyz}" izz="${lift_base_link_izz}"/>
         </inertia>
         <visual>
           <geometry>
-            <box size="0.220 0.200 0.015"/>
+            <box size="${base_box_size}"/>
           </geometry>
           <material name="gray"/>
@@ -73,5 +130,5 @@
         <collision>
           <geometry>
-            <box size="0.220 0.200 0.015"/>
+            <box size="${base_box_size}"/>
           </geometry>
         </collision>
@@ -81,10 +138,10 @@
     <link name="${tf_prefix}ewellix_lift_lower_link">
       <inertia>
-        <mass value="1.9521070e+01"/>
-        <inertia ixx="0.46604111" ixy="0" ixz="0" iyy="0.46480515" iyz="-0.002668667" izz="0.1561"/>
+        <mass value="${lower_mass_value}"/>
+        <inertia ixx="${lift_lower_link_ixx}" ixy="${lift_lower_link_ixy}" ixz="${lift_lower_link_ixz}" iyy="${lift_lower_link_iyy}" iyz="${lift_lower_link_iyz}" izz="${lift_lower_link_izz}"/>
       </inertia>
       <visual>
         <geometry>
-          <mesh filename= "package://ewellix_liftkit_description/meshes/visual/lift_low.dae"/>
+          <mesh filename= "${lower_mesh_filename}"/>
         </geometry>
         <material name="gray"/>
@@ -92,5 +149,5 @@
       <collision>
         <geometry>
-          <box size="0.163 0.163 0.575"/>
+          <box size="${lower_box_size}"/>
         </geometry>
       </collision>
@@ -107,10 +164,10 @@
     <link name="${tf_prefix}ewellix_lift_middle_link">
       <inertia>
-        <mass value="1.5593303e+01"/>
-        <inertia ixx="0.34930648" ixy="0" ixz="0" iyy="0.34930648" iyz="0" izz="0.095393471"/>
+        <mass value="${middle_mass_value}"/>
+        <inertia ixx="${lift_middle_link_ixx}" ixy="${lift_middle_link_ixy}" ixz="${lift_middle_link_ixz}" iyy="${lift_middle_link_iyy}" iyz="${lift_middle_link_iyz}" izz="${lift_middle_link_izz}"/>
       </inertia>
       <visual>
         <geometry>
-          <mesh filename= "package://ewellix_liftkit_description/meshes/visual/lift_mid.dae"/>
+          <mesh filename= "${middle_mesh_filename}"/>
         </geometry>
         <material name="gray"/>
@@ -118,5 +175,5 @@
       <collision>
         <geometry>
-          <box size="0.146 0.146 0.483"/>
+          <box size="${middle_box_size}"/>
         </geometry>
       </collision>
@@ -125,10 +182,10 @@
     <link name="${tf_prefix}ewellix_lift_higher_link">
       <inertia>
-        <mass value="1.5166778e+01"/>
-        <inertia ixx="0.35552099" ixy="9.6314989e-6" ixz="2.284786e-5" iyy="0.35552876" iyz="5.4910201e-5" izz="0.069925583"/>
+        <mass value="${higher_mass_value}"/>
+        <inertia ixx="${lift_higher_link_ixx}" ixy="${lift_higher_link_ixy}" ixz="${lift_higher_link_ixz}" iyy="${lift_higher_link_iyy}" iyz="${lift_higher_link_iyz}" izz="${lift_higher_link_izz}"/>
       </inertia>
       <visual>
         <geometry>
-          <mesh filename= "package://ewellix_liftkit_description/meshes/visual/lift_high.dae"/>
+          <mesh filename= "${higher_mesh_filename}"/>
         </geometry>
         <material name="gray"/>
@@ -136,5 +193,5 @@
       <collision>
         <geometry>
-          <box size="0.129 0.129 0.488"/>
+          <box size="${higher_box_size}"/>
         </geometry>
       </collision>
@@ -162,10 +219,10 @@
       <link name="${tf_prefix}ewellix_lift_top_link">
         <inertia>
-          <mass value="4.9139525"/>
-          <inertia ixx="0.02015548" ixy="-2.281101e-5" ixz="0" iyy="0.01664141" iyz="0" izz="0.03661307"/>
+          <mass value="${top_mass_value}"/>
+          <inertia ixx="${lift_top_link_ixx}" ixy="${lift_top_link_ixy}" ixz="${lift_top_link_ixz}" iyy="${lift_top_link_iyy}" iyz="${lift_top_link_iyz}" izz="${lift_top_link_izz}"/>
         </inertia>
         <visual>
           <geometry>
-            <box size="0.200 0.220 0.015"/>
+            <box size="${top_box_size}"/>
           </geometry>
           <material name="gray"/>
@@ -173,5 +230,5 @@
         <collision>
           <geometry>
-            <box size="0.200 0.220 0.015"/>
+            <box size="${top_box_size}"/>
           </geometry>
         </collision>

Commit message: Placed inertia/mass values in for 500 mm, as well as mesh files. Initial test for 500 mm xacro was successful. Needs cleaning.

File: ewellix_liftkit_description/urdf/ewellix_lift.xacro (robot description, xacro)
@@ -8,4 +8,5 @@
     omit_plates:=false
     is_700:=true
+    is_500:=true
     use_fake_hardware:=false
     com_port:=/dev/ttyUSB0
@@ -18,4 +19,5 @@
     </xacro:if>
     <xacro:if value="${is_700}">
+    <xacro:property name="height_limit" value="0.7"/>
     <xacro:property name="base_mass_value" value="1.7383784"/>
     <xacro:property name="base_box_size" value="0.220 0.200 0.015"/>
@@ -26,4 +28,5 @@
     <xacro:property name="lift_base_link_iyz" value="0.0" scope="parent"/>
     <xacro:property name="lift_base_link_izz" value="1.2717018e-02" scope="parent"/>
+    <xacro:property name="base_to_lower_origin_z" value="0.295"/>
     <xacro:property name="lower_mass_value" value="1.9521070e+01"/>
     <xacro:property name="lower_box_size" value="0.163 0.163 0.575"/>
@@ -62,50 +65,52 @@
     <xacro:property name="lift_top_link_izz" value="0.03661307" scope="parent"/>
     </xacro:if>
-     <!--
-    <xacro:if value="500">
-    <xacro:property name="base_mass_value" value="0.0"/>
-    <xacro:property name="base_box_size" value="0.0 0.0 0.0"/>
-    <xacro:property name="lift_base_link_ixx" value="0.0" scope="parent"/>
+    <!-- <xacro:if value="${is_500}">
+    <xacro:property name="height_limit" value="0.5"/>
+    <xacro:property name="base_mass_value" value="1.7383784"/>
+    <xacro:property name="base_box_size" value="0.220 0.200 0.015"/>
+    <xacro:property name="lift_base_link_ixx" value="5.7788740E-03" scope="parent"/>
     <xacro:property name="lift_base_link_ixy" value="0.0" scope="parent"/>
     <xacro:property name="lift_base_link_ixz" value="0.0" scope="parent"/>
-    <xacro:property name="lift_base_link_iyy" value="0.0" scope="parent"/>
+    <xacro:property name="lift_base_link_iyy" value="1.2717010E-02" scope="parent"/>
     <xacro:property name="lift_base_link_iyz" value="0.0" scope="parent"/>
-    <xacro:property name="lift_base_link_izz" value="0.0" scope="parent"/>
-    <xacro:property name="lower_mass_value" value="0.0"/>
-    <xacro:property name="lower_box_size" value="0.0 0.0 0.0"/>
-    <xacro:property name="lower_mesh_filename" value="..."/>
-    <xacro:property name="lift_lower_link_ixx" value="0.0" scope="parent"/>
+    <xacro:property name="lift_base_link_izz" value="7.0031710E-03" scope="parent"/>
+    <xacro:property name="base_to_lower_origin_z" value="0.2532"/>
+    <xacro:property name="lower_mass_value" value="6.746306"/>
+    <xacro:property name="lower_box_size" value="0.163 0.163 0.4764"/>
+    <xacro:property name="lower_mesh_filename" value="package://ewellix_liftkit_description/meshes/visual/lift_low_500mm.stl"/>
+    <xacro:property name="lift_lower_link_ixx" value="1.577769E-07" scope="parent"/>
     <xacro:property name="lift_lower_link_ixy" value="0.0" scope="parent"/>
     <xacro:property name="lift_lower_link_ixz" value="0.0" scope="parent"/>
-    <xacro:property name="lift_lower_link_iyy" value="0.0" scope="parent"/>
-    <xacro:property name="lift_lower_link_iyz" value="0.0" scope="parent"/>
-    <xacro:property name="lift_lower_link_izz" value="0.0" scope="parent"/>
-    <xacro:property name="middle_mass_value" value="0.0"/>
-    <xacro:property name="middle_box_size" value="0.0 0.0 0.0"/>
-    <xacro:property name="middle_mesh_filename" value="..."/>
-    <xacro:property name="lift_middle_link_ixx" value="0.0" scope="parent"/>
+    <xacro:property name="lift_lower_link_iyy" value="5.379943E-08" scope="parent"/>
+    <xacro:property name="lift_lower_link_iyz" value="1.521466E-10" scope="parent"/>
+    <xacro:property name="lift_lower_link_izz" value="1.577222E-07" scope="parent"/>
+    <xacro:property name="middle_mass_value" value="5.411604"/>
+    <xacro:property name="middle_box_size" value="0.146 0.146 0.4794"/>
+    <xacro:property name="middle_mesh_filename" value="package://ewellix_liftkit_description/meshes/visual/lift_mid_500mm.stl"/>
+    <xacro:property name="lift_middle_link_ixx" value="1.196271E-01" scope="parent"/>
     <xacro:property name="lift_middle_link_ixy" value="0.0" scope="parent"/>
     <xacro:property name="lift_middle_link_ixz" value="0.0" scope="parent"/>
-    <xacro:property name="lift_middle_link_iyy" value="0.0" scope="parent"/>
+    <xacro:property name="lift_middle_link_iyy" value="3.309969E-02" scope="parent"/>
     <xacro:property name="lift_middle_link_iyz" value="0.0" scope="parent"/>
-    <xacro:property name="lift_middle_link_izz" value="0.0" scope="parent"/>
-    <xacro:property name="higher_mass_value" value="0.0"/>
-    <xacro:property name="higher_box_size" value="0.0 0.0 0.0"/>
-    <xacro:property name="higher_mesh_filename" value="..."/>
-    <xacro:property name="lift_higher_link_ixx" value="0.0" scope="parent"/>
-    <xacro:property name="lift_higher_link_ixy" value="0.0" scope="parent"/>
-    <xacro:property name="lift_higher_link_ixz" value="0.0" scope="parent"/>
-    <xacro:property name="lift_higher_link_iyy" value="0.0" scope="parent"/>
-    <xacro:property name="lift_higher_link_iyz" value="0.0" scope="parent"/>
-    <xacro:property name="lift_higher_link_izz" value="0.0" scope="parent"/>
-    <xacro:property name="lift_top_link_ixx" value="0.0" scope="parent"/>
-    <xacro:property name="lift_top_link_ixy" value="0.0" scope="parent"/>
-    <xacro:property name="lift_top_link_ixz" value="0.0" scope="parent"/>
-    <xacro:property name="lift_top_link_iyy" value="0.0" scope="parent"/>
-    <xacro:property name="lift_top_link_iyz" value="0.0" scope="parent"/>
-    <xacro:property name="lift_top_link_izz" value="0.0" scope="parent"/>
-    </xacro:if>
-    -->
-    <xacro:unless value="${not omit_plates}">
+    <xacro:property name="lift_middle_link_izz" value="1.196271E-01" scope="parent"/>
+    <xacro:property name="higher_mass_value" value="5.324879"/>
+    <xacro:property name="higher_box_size" value="0.129 0.129 0.490"/>
+    <xacro:property name="higher_mesh_filename" value="package://ewellix_liftkit_description/meshes/visual/lift_high_500mm.stl"/>
+    <xacro:property name="lift_higher_link_ixx" value="1.253755E-01" scope="parent"/>
+    <xacro:property name="lift_higher_link_ixy" value="-1.864377E-05" scope="parent"/>
+    <xacro:property name="lift_higher_link_ixz" value="3.368651E-06" scope="parent"/>
+    <xacro:property name="lift_higher_link_iyy" value="2.455221E-02" scope="parent"/>
+    <xacro:property name="lift_higher_link_iyz" value="-7.757573E-06" scope="parent"/>
+    <xacro:property name="lift_higher_link_izz" value="1.253728E-01" scope="parent"/>
+    <xacro:property name="top_mass_value" value="1.718423"/>
+    <xacro:property name="top_box_size" value="0.200 0.220 0.015"/>
+    <xacro:property name="lift_top_link_ixx" value="5.819538E-03" scope="parent"/>
+    <xacro:property name="lift_top_link_ixy" value="4.555714E-09" scope="parent"/>
+    <xacro:property name="lift_top_link_ixz" value="8.002694E-06" scope="parent"/>
+    <xacro:property name="lift_top_link_iyy" value="1.280362E-02" scope="parent"/>
+    <xacro:property name="lift_top_link_iyz" value="1.967468E-09" scope="parent"/>
+    <xacro:property name="lift_top_link_izz" value="7.048366E-03" scope="parent"/>
+    </xacro:if> -->
+  <xacro:unless value="${not omit_plates}">
       <xacro:property name="lift_base_link_name" value="${tf_prefix}ewellix_lift_lower_link"/>
     </xacro:unless>
@@ -158,5 +163,5 @@
         <parent link="${tf_prefix}ewellix_lift_base_link"/>
         <child link="${tf_prefix}ewellix_lift_lower_link"/>
-        <origin xyz="0 0 0.295" rpy="0 0 0"/>
+        <origin xyz="0 0 ${base_to_lower_origin_z}" rpy="0 0 0"/>
       </joint>
     </xacro:if>

Commit message: Modified the base_to_origin_z value in the 500mm xacro if-block. (Equation = origin of lower tier z val + 1/2(depth of base)). Currently the visual looks good, but the lower collision object is floating wrt to the base. Need to revisit.

File: ewellix_liftkit_description/urdf/ewellix_lift.xacro (robot description, xacro)
@@ -8,5 +8,5 @@
     omit_plates:=false
     is_700:=true
-    is_500:=true
+    is_500:=false
     use_fake_hardware:=false
     com_port:=/dev/ttyUSB0
@@ -65,5 +65,5 @@
     <xacro:property name="lift_top_link_izz" value="0.03661307" scope="parent"/>
     </xacro:if>
-    <!-- <xacro:if value="${is_500}">
+    <xacro:if value="${is_500}">
     <xacro:property name="height_limit" value="0.5"/>
     <xacro:property name="base_mass_value" value="1.7383784"/>
@@ -75,7 +75,7 @@
     <xacro:property name="lift_base_link_iyz" value="0.0" scope="parent"/>
     <xacro:property name="lift_base_link_izz" value="7.0031710E-03" scope="parent"/>
-    <xacro:property name="base_to_lower_origin_z" value="0.2532"/>
+    <xacro:property name="base_to_lower_origin_z" value="0.2645"/>
     <xacro:property name="lower_mass_value" value="6.746306"/>
-    <xacro:property name="lower_box_size" value="0.163 0.163 0.4764"/>
+    <xacro:property name="lower_box_size" value="0.163 0.163 0.4744"/>
     <xacro:property name="lower_mesh_filename" value="package://ewellix_liftkit_description/meshes/visual/lift_low_500mm.stl"/>
     <xacro:property name="lift_lower_link_ixx" value="1.577769E-07" scope="parent"/>
@@ -111,5 +111,5 @@
     <xacro:property name="lift_top_link_iyz" value="1.967468E-09" scope="parent"/>
     <xacro:property name="lift_top_link_izz" value="7.048366E-03" scope="parent"/>
-    </xacro:if> -->
+    </xacro:if>
   <xacro:unless value="${not omit_plates}">
       <xacro:property name="lift_base_link_name" value="${tf_prefix}ewellix_lift_lower_link"/>

Commit message: Fixed lower tier mesh origin issue. Recentered it. Corrected some vals.

File: ewellix_liftkit_description/urdf/ewellix_lift.xacro (robot description, xacro)
@@ -7,6 +7,6 @@
     height_limit:=0.7
     omit_plates:=false
-    is_700:=true
-    is_500:=false
+    is_700:=false
+    is_500:=true
     use_fake_hardware:=false
     com_port:=/dev/ttyUSB0
@@ -75,7 +75,7 @@
     <xacro:property name="lift_base_link_iyz" value="0.0" scope="parent"/>
     <xacro:property name="lift_base_link_izz" value="7.0031710E-03" scope="parent"/>
-    <xacro:property name="base_to_lower_origin_z" value="0.2645"/>
+    <xacro:property name="base_to_lower_origin_z" value="0.2382"/>
     <xacro:property name="lower_mass_value" value="6.746306"/>
-    <xacro:property name="lower_box_size" value="0.163 0.163 0.4744"/>
+    <xacro:property name="lower_box_size" value="0.163 0.163 0.4764"/>
     <xacro:property name="lower_mesh_filename" value="package://ewellix_liftkit_description/meshes/visual/lift_low_500mm.stl"/>
     <xacro:property name="lift_lower_link_ixx" value="1.577769E-07" scope="parent"/>
