Commit message: Restructured the origin to origin z-position values to be parameters defined in the if blocks initially. Because the vals are different for each of the liftkit types. To note: I only moved the 700 mm stroke (default) values as they were. NO VALUES FOR 700mm STROKE LIFTKIT HAS CHANGED. I only calculated and modified the 500 mm values and moved around the 700 mm stroke values (DEFAULT) around in a way which it was not affected. Formula I used to calculate origin to origin distance = 1/2(height of tier) + 1/2(height of other tier). For distance betweeen origin of tier and origin of base = 1/2(height of tier) + 1/2(height of base). Insert height of tier or base you want to compare.

File: ewellix_liftkit_description/urdf/ewellix_lift.xacro (robot description, xacro)
@@ -38,4 +38,5 @@
       <xacro:property name="lift_lower_link_iyz" value="-0.002668667" scope="parent"/>
       <xacro:property name="lift_lower_link_izz" value="0.1561" scope="parent"/>
+      <xacro:property name="lower_to_higher_origin_z" value="0.0915"/>
       <xacro:property name="middle_mass_value" value="1.5593303e+01"/>
       <xacro:property name="middle_box_size" value="0.146 0.146 0.483"/>
@@ -47,4 +48,5 @@
       <xacro:property name="lift_middle_link_iyz" value="0.0" scope="parent"/>
       <xacro:property name="lift_middle_link_izz" value="0.095393471" scope="parent"/>
+      <xacro:property name="middle_to_higher_origin_z" value="-0.03397"/>
       <xacro:property name="higher_mass_value" value="1.5166778e+01"/>
       <xacro:property name="higher_box_size" value="0.129 0.129 0.488"/>
@@ -56,4 +58,5 @@
       <xacro:property name="lift_higher_link_iyz" value="5.4910201e-5" scope="parent"/>
       <xacro:property name="lift_higher_link_izz" value="0.069925583" scope="parent"/>
+      <xacro:property name="higher_to_top_origin_z" value="0.2515"/>
       <xacro:property name="top_mass_value" value="4.9139525"/>
       <xacro:property name="top_box_size" value="0.200 0.220 0.015"/>
@@ -64,4 +67,5 @@
       <xacro:property name="lift_top_link_iyz" value="0.0" scope="parent"/>
       <xacro:property name="lift_top_link_izz" value="0.03661307" scope="parent"/>
+      <xacro:property name="lift_tip_joint_origin_z" value="0.244"/>
     </xacro:if>
     <!--For 500 mm stroke-->
@@ -79,5 +83,5 @@
       <xacro:property name="lift_base_link_iyz" value="0.0" scope="parent"/>
       <xacro:property name="lift_base_link_izz" value="7.0031710E-03" scope="parent"/>
-      <xacro:property name="base_to_lower_origin_z" value="0.2382"/>
+      <xacro:property name="base_to_lower_origin_z" value="0.2457"/>
       <xacro:property name="lower_mass_value" value="6.746306"/>
       <xacro:property name="lower_box_size" value="0.163 0.163 0.4764"/>
@@ -89,4 +93,5 @@
       <xacro:property name="lift_lower_link_iyz" value="1.521466E-10" scope="parent"/>
       <xacro:property name="lift_lower_link_izz" value="1.577222E-07" scope="parent"/>
+      <xacro:property name="lower_to_higher_origin_z" value="0.0068"/>
       <xacro:property name="middle_mass_value" value="5.411604"/>
       <xacro:property name="middle_box_size" value="0.146 0.146 0.4794"/>
@@ -98,4 +103,5 @@
       <xacro:property name="lift_middle_link_iyz" value="0.0" scope="parent"/>
       <xacro:property name="lift_middle_link_izz" value="1.196271E-01" scope="parent"/>
+      <xacro:property name="middle_to_higher_origin_z" value="-0.0053"/>
       <xacro:property name="higher_mass_value" value="5.324879"/>
       <xacro:property name="higher_box_size" value="0.129 0.129 0.490"/>
@@ -107,4 +113,5 @@
       <xacro:property name="lift_higher_link_iyz" value="-7.757573E-06" scope="parent"/>
       <xacro:property name="lift_higher_link_izz" value="1.253728E-01" scope="parent"/>
+      <xacro:property name="higher_to_top_origin_z" value="0.2525"/>
       <xacro:property name="top_mass_value" value="1.718423"/>
       <xacro:property name="top_box_size" value="0.200 0.220 0.015"/>
@@ -115,4 +122,5 @@
       <xacro:property name="lift_top_link_iyz" value="1.967468E-09" scope="parent"/>
       <xacro:property name="lift_top_link_izz" value="7.048366E-03" scope="parent"/>
+      <xacro:property name="lift_tip_joint_origin_z" value="0.245"/>
     </xacro:if>
   <xacro:unless value="${not omit_plates}">
@@ -211,5 +219,5 @@
       <parent link="${tf_prefix}ewellix_lift_lower_link"/>
       <child link="${tf_prefix}ewellix_lift_higher_link"/>
-      <origin xyz="0 0 0.0915" rpy="0 0 0"/>
+      <origin xyz="0 0 ${lower_to_higher_origin_z}" rpy="0 0 0"/>
       <axis xyz="0 0 1"/>
       <limit lower="0" upper="${height_limit}" effort="1000" velocity="1"/>
@@ -219,5 +227,5 @@
       <parent link="${tf_prefix}ewellix_lift_higher_link"/>
       <child link="${tf_prefix}ewellix_lift_middle_link"/>
-      <origin xyz="0 0 -0.03397" rpy="0 0 0"/>
+      <origin xyz="0 0 ${middle_to_higher_origin_z}" rpy="0 0 0"/>
       <axis xyz="0 0 -1"/>
       <limit lower="0" upper="0.351" effort="1000" velocity="1"/>
@@ -249,5 +257,5 @@
         <parent link="${tf_prefix}ewellix_lift_higher_link"/>
         <child link="${tf_prefix}ewellix_lift_top_link"/>
-        <origin xyz="0 0 0.2515" rpy="0 0 0"/>
+        <origin xyz="0 0 ${higher_to_top_origin_z}" rpy="0 0 0"/>
       </joint>
     </xacro:if>
@@ -256,5 +264,5 @@
       <parent link="${tf_prefix}ewellix_lift_higher_link"/>
       <child link="${tf_prefix}ewellix_lift_tip_link"/>
-      <origin xyz="0 0 0.244" rpy="0 0 0"/>
+      <origin xyz="0 0 ${lift_tip_joint_origin_z}" rpy="0 0 0"/>
     </joint>
     <xacro:include filename="$(find ewellix_liftkit_description)/urdf/ewellix_liftkit.ros2_control.xacro" />

Commit message: Changed name of 700mm meshes for consistency.

File: ewellix_liftkit_description/urdf/ewellix_lift.xacro (robot description, xacro)
@@ -31,5 +31,5 @@
       <xacro:property name="lower_mass_value" value="1.9521070e+01"/>
       <xacro:property name="lower_box_size" value="0.163 0.163 0.575"/>
-      <xacro:property name="lower_mesh_filename" value="package://ewellix_liftkit_description/meshes/visual/lift_low.dae"/>
+      <xacro:property name="lower_mesh_filename" value="package://ewellix_liftkit_description/meshes/visual/lift_low_700mm.dae"/>
       <xacro:property name="lift_lower_link_ixx" value="0.46604111" scope="parent"/>
       <xacro:property name="lift_lower_link_ixy" value="0.0" scope="parent"/>
@@ -41,5 +41,5 @@
       <xacro:property name="middle_mass_value" value="1.5593303e+01"/>
       <xacro:property name="middle_box_size" value="0.146 0.146 0.483"/>
-      <xacro:property name="middle_mesh_filename" value="package://ewellix_liftkit_description/meshes/visual/lift_mid.dae"/>
+      <xacro:property name="middle_mesh_filename" value="package://ewellix_liftkit_description/meshes/visual/lift_mid_700mm.dae"/>
       <xacro:property name="lift_middle_link_ixx" value="0.34930648" scope="parent"/>
       <xacro:property name="lift_middle_link_ixy" value="0.0" scope="parent"/>
@@ -51,5 +51,5 @@
       <xacro:property name="higher_mass_value" value="1.5166778e+01"/>
       <xacro:property name="higher_box_size" value="0.129 0.129 0.488"/>
-      <xacro:property name="higher_mesh_filename" value="package://ewellix_liftkit_description/meshes/visual/lift_high.dae"/>
+      <xacro:property name="higher_mesh_filename" value="package://ewellix_liftkit_description/meshes/visual/lift_high_700mm.dae"/>
       <xacro:property name="lift_higher_link_ixx" value="0.35552099" scope="parent"/>
       <xacro:property name="lift_higher_link_ixy" value="9.6314989e-6" scope="parent"/>

Commit message: Added the statement so height_limit caps of at 0.7m.

File: ewellix_liftkit_description/urdf/ewellix_lift.xacro (robot description, xacro)
@@ -20,4 +20,7 @@
     <!--For 700 mm stroke-->
     <xacro:if value="${is_700}">
+      <xacro:if value="$(eval height_limit >= 0.7)">
+        <xacro:property name="height_limit" value="0.7"/>
+      </xacro:if>
       <xacro:property name="base_mass_value" value="1.7383784"/>
       <xacro:property name="base_box_size" value="0.220 0.200 0.015"/>

Commit message: Made the middle tier upper limit a param bc it's different for each liftkit type.

File: ewellix_liftkit_description/urdf/ewellix_lift.xacro (robot description, xacro)
@@ -50,4 +50,5 @@
       <xacro:property name="lift_middle_link_izz" value="0.095393471" scope="parent"/>
       <xacro:property name="middle_to_higher_origin_z" value="-0.03397"/>
+      <xacro:property name="middle_upper_limit" value="0.351"/>
       <xacro:property name="higher_mass_value" value="1.5166778e+01"/>
       <xacro:property name="higher_box_size" value="0.129 0.129 0.488"/>
@@ -105,4 +106,5 @@
       <xacro:property name="lift_middle_link_izz" value="1.196271E-01" scope="parent"/>
       <xacro:property name="middle_to_higher_origin_z" value="-0.0053"/>
+      <xacro:property name="middle_upper_limit" value="0.25"/>
       <xacro:property name="higher_mass_value" value="5.324879"/>
       <xacro:property name="higher_box_size" value="0.129 0.129 0.490"/>
@@ -229,5 +231,5 @@
       <origin xyz="0 0 ${middle_to_higher_origin_z}" rpy="0 0 0"/>
       <axis xyz="0 0 -1"/>
-      <limit lower="0" upper="0.351" effort="1000" velocity="1"/>
+      <limit lower="0" upper="${middle_upper_limit}" effort="1000" velocity="1"/>
       <mimic joint="${tf_prefix}ewellix_lift_lower_to_higher" multiplier="0.5" offset="0"/>
     </joint>

Commit message: Modified values for 700 mm stroke liftkit. Removed scientific notation

File: ewellix_liftkit_description/urdf/ewellix_lift.xacro (robot description, xacro)
@@ -23,50 +23,50 @@
       <xacro:property name="base_mass_value" value="1.7383784"/>
       <xacro:property name="base_box_size" value="0.220 0.200 0.015"/>
-      <xacro:property name="lift_base_link_ixx" value="5.7788770e-03" scope="parent"/>
+      <xacro:property name="lift_base_link_ixx" value="0.00577887" scope="parent"/>
       <xacro:property name="lift_base_link_ixy" value="0.0" scope="parent"/>
       <xacro:property name="lift_base_link_ixz" value="0.0" scope="parent"/>
-      <xacro:property name="lift_base_link_iyy" value="7.0031715e-03" scope="parent"/>
+      <xacro:property name="lift_base_link_iyy" value="0.01271701" scope="parent"/>
       <xacro:property name="lift_base_link_iyz" value="0.0" scope="parent"/>
-      <xacro:property name="lift_base_link_izz" value="1.2717018e-02" scope="parent"/>
+      <xacro:property name="lift_base_link_izz" value="0.00700317" scope="parent"/>
       <xacro:property name="base_to_lower_origin_z" value="0.295"/>
-      <xacro:property name="lower_mass_value" value="1.9521070e+01"/>
+      <xacro:property name="lower_mass_value" value="8.176405"/>
       <xacro:property name="lower_box_size" value="0.163 0.163 0.575"/>
       <xacro:property name="lower_mesh_filename" value="package://ewellix_liftkit_description/meshes/visual/lift_low_700mm.dae"/>
-      <xacro:property name="lift_lower_link_ixx" value="0.46604111" scope="parent"/>
+      <xacro:property name="lift_lower_link_ixx" value="0.26551310" scope="parent"/>
       <xacro:property name="lift_lower_link_ixy" value="0.0" scope="parent"/>
       <xacro:property name="lift_lower_link_ixz" value="0.0" scope="parent"/>
-      <xacro:property name="lift_lower_link_iyy" value="0.46480515" scope="parent"/>
-      <xacro:property name="lift_lower_link_iyz" value="-0.002668667" scope="parent"/>
-      <xacro:property name="lift_lower_link_izz" value="0.1561" scope="parent"/>
+      <xacro:property name="lift_lower_link_iyy" value="0.06547122" scope="parent"/>
+      <xacro:property name="lift_lower_link_iyz" value="0.00111055" scope="parent"/>
+      <xacro:property name="lift_lower_link_izz" value="0.26508300" scope="parent"/>
       <xacro:property name="lower_to_higher_origin_z" value="0.0915"/>
-      <xacro:property name="middle_mass_value" value="1.5593303e+01"/>
+      <xacro:property name="middle_mass_value" value="6.54457"/>
       <xacro:property name="middle_box_size" value="0.146 0.146 0.483"/>
       <xacro:property name="middle_mesh_filename" value="package://ewellix_liftkit_description/meshes/visual/lift_mid_700mm.dae"/>
-      <xacro:property name="lift_middle_link_ixx" value="0.34930648" scope="parent"/>
+      <xacro:property name="lift_middle_link_ixx" value="0.20223860" scope="parent"/>
       <xacro:property name="lift_middle_link_ixy" value="0.0" scope="parent"/>
       <xacro:property name="lift_middle_link_ixz" value="0.0" scope="parent"/>
-      <xacro:property name="lift_middle_link_iyy" value="0.34930648" scope="parent"/>
+      <xacro:property name="lift_middle_link_iyy" value="0.04003302" scope="parent"/>
       <xacro:property name="lift_middle_link_iyz" value="0.0" scope="parent"/>
-      <xacro:property name="lift_middle_link_izz" value="0.095393471" scope="parent"/>
+      <xacro:property name="lift_middle_link_izz" value="0.20223860" scope="parent"/>
       <xacro:property name="middle_to_higher_origin_z" value="-0.03397"/>
       <xacro:property name="middle_upper_limit" value="0.351"/>
-      <xacro:property name="higher_mass_value" value="1.5166778e+01"/>
+      <xacro:property name="higher_mass_value" value="6.375617"/>
       <xacro:property name="higher_box_size" value="0.129 0.129 0.488"/>
       <xacro:property name="higher_mesh_filename" value="package://ewellix_liftkit_description/meshes/visual/lift_high_700mm.dae"/>
-      <xacro:property name="lift_higher_link_ixx" value="0.35552099" scope="parent"/>
-      <xacro:property name="lift_higher_link_ixy" value="9.6314989e-6" scope="parent"/>
-      <xacro:property name="lift_higher_link_ixz" value="2.284786e-5" scope="parent"/>
-      <xacro:property name="lift_higher_link_iyy" value="0.35552876" scope="parent"/>
-      <xacro:property name="lift_higher_link_iyz" value="5.4910201e-5" scope="parent"/>
-      <xacro:property name="lift_higher_link_izz" value="0.069925583" scope="parent"/>
+      <xacro:property name="lift_higher_link_ixx" value="0.20932400" scope="parent"/>
+      <xacro:property name="lift_higher_link_ixy" value="-0.00002260" scope="parent"/>
+      <xacro:property name="lift_higher_link_ixz" value="0.00000337" scope="parent"/>
+      <xacro:property name="lift_higher_link_iyy" value="0.02950402" scope="parent"/>
+      <xacro:property name="lift_higher_link_iyz" value="-0.00000940" scope="parent"/>
+      <xacro:property name="lift_higher_link_izz" value="0.20932130" scope="parent"/>
       <xacro:property name="higher_to_top_origin_z" value="0.2515"/>
-      <xacro:property name="top_mass_value" value="4.9139525"/>
+      <xacro:property name="top_mass_value" value="1.718423"/>
       <xacro:property name="top_box_size" value="0.200 0.220 0.015"/>
-      <xacro:property name="lift_top_link_ixx" value="0.02015548" scope="parent"/>
-      <xacro:property name="lift_top_link_ixy" value="-2.281101e-5" scope="parent"/>
-      <xacro:property name="lift_top_link_ixz" value="0.0" scope="parent"/>
-      <xacro:property name="lift_top_link_iyy" value="0.01664141" scope="parent"/>
-      <xacro:property name="lift_top_link_iyz" value="0.0" scope="parent"/>
-      <xacro:property name="lift_top_link_izz" value="0.03661307" scope="parent"/>
+      <xacro:property name="lift_top_link_ixx" value="0.00581954" scope="parent"/>
+      <xacro:property name="lift_top_link_ixy" value="0.00000000" scope="parent"/>
+      <xacro:property name="lift_top_link_ixz" value="0.00000800" scope="parent"/>
+      <xacro:property name="lift_top_link_iyy" value="0.01280362" scope="parent"/>
+      <xacro:property name="lift_top_link_iyz" value="0.00000000" scope="parent"/>
+      <xacro:property name="lift_top_link_izz" value="0.00704837" scope="parent"/>
       <xacro:property name="lift_tip_joint_origin_z" value="0.244"/>
     </xacro:if>
@@ -79,30 +79,30 @@
       <xacro:property name="base_mass_value" value="1.7383784"/>
       <xacro:property name="base_box_size" value="0.220 0.200 0.015"/>
-      <xacro:property name="lift_base_link_ixx" value="5.7788740E-03" scope="parent"/>
+      <xacro:property name="lift_base_link_ixx" value="0.00577887" scope="parent"/>
       <xacro:property name="lift_base_link_ixy" value="0.0" scope="parent"/>
       <xacro:property name="lift_base_link_ixz" value="0.0" scope="parent"/>
-      <xacro:property name="lift_base_link_iyy" value="1.2717010E-02" scope="parent"/>
+      <xacro:property name="lift_base_link_iyy" value="0.01271701" scope="parent"/>
       <xacro:property name="lift_base_link_iyz" value="0.0" scope="parent"/>
-      <xacro:property name="lift_base_link_izz" value="7.0031710E-03" scope="parent"/>
+      <xacro:property name="lift_base_link_izz" value="0.00700317" scope="parent"/>
       <xacro:property name="base_to_lower_origin_z" value="0.2457"/>
       <xacro:property name="lower_mass_value" value="6.746306"/>
       <xacro:property name="lower_box_size" value="0.163 0.163 0.4764"/>
       <xacro:property name="lower_mesh_filename" value="package://ewellix_liftkit_description/meshes/visual/lift_low_500mm.stl"/>
-      <xacro:property name="lift_lower_link_ixx" value="1.577769E-07" scope="parent"/>
+      <xacro:property name="lift_lower_link_ixx" value="0.00000016" scope="parent"/>
       <xacro:property name="lift_lower_link_ixy" value="0.0" scope="parent"/>
       <xacro:property name="lift_lower_link_ixz" value="0.0" scope="parent"/>
-      <xacro:property name="lift_lower_link_iyy" value="5.379943E-08" scope="parent"/>
-      <xacro:property name="lift_lower_link_iyz" value="1.521466E-10" scope="parent"/>
-      <xacro:property name="lift_lower_link_izz" value="1.577222E-07" scope="parent"/>
+      <xacro:property name="lift_lower_link_iyy" value="0.00000005" scope="parent"/>
+      <xacro:property name="lift_lower_link_iyz" value="0.0" scope="parent"/>
+      <xacro:property name="lift_lower_link_izz" value="0.00000016" scope="parent"/>
       <xacro:property name="lower_to_higher_origin_z" value="0.0068"/>
       <xacro:property name="middle_mass_value" value="5.411604"/>
       <xacro:property name="middle_box_size" value="0.146 0.146 0.4794"/>
       <xacro:property name="middle_mesh_filename" value="package://ewellix_liftkit_description/meshes/visual/lift_mid_500mm.stl"/>
-      <xacro:property name="lift_middle_link_ixx" value="1.196271E-01" scope="parent"/>
+      <xacro:property name="lift_middle_link_ixx" value="0.11962710" scope="parent"/>
       <xacro:property name="lift_middle_link_ixy" value="0.0" scope="parent"/>
       <xacro:property name="lift_middle_link_ixz" value="0.0" scope="parent"/>
-      <xacro:property name="lift_middle_link_iyy" value="3.309969E-02" scope="parent"/>
+      <xacro:property name="lift_middle_link_iyy" value="0.03309969" scope="parent"/>
       <xacro:property name="lift_middle_link_iyz" value="0.0" scope="parent"/>
-      <xacro:property name="lift_middle_link_izz" value="1.196271E-01" scope="parent"/>
+      <xacro:property name="lift_middle_link_izz" value="0.11962710" scope="parent"/>
       <xacro:property name="middle_to_higher_origin_z" value="-0.0053"/>
       <xacro:property name="middle_upper_limit" value="0.25"/>
@@ -110,19 +110,19 @@
       <xacro:property name="higher_box_size" value="0.129 0.129 0.490"/>
       <xacro:property name="higher_mesh_filename" value="package://ewellix_liftkit_description/meshes/visual/lift_high_500mm.stl"/>
-      <xacro:property name="lift_higher_link_ixx" value="1.253755E-01" scope="parent"/>
-      <xacro:property name="lift_higher_link_ixy" value="-1.864377E-05" scope="parent"/>
-      <xacro:property name="lift_higher_link_ixz" value="3.368651E-06" scope="parent"/>
-      <xacro:property name="lift_higher_link_iyy" value="2.455221E-02" scope="parent"/>
-      <xacro:property name="lift_higher_link_iyz" value="-7.757573E-06" scope="parent"/>
-      <xacro:property name="lift_higher_link_izz" value="1.253728E-01" scope="parent"/>
+      <xacro:property name="lift_higher_link_ixx" value="0.12537550" scope="parent"/>
+      <xacro:property name="lift_higher_link_ixy" value="-0.00001864" scope="parent"/>
+      <xacro:property name="lift_higher_link_ixz" value="0.00000337" scope="parent"/>
+      <xacro:property name="lift_higher_link_iyy" value="0.02455221" scope="parent"/>
+      <xacro:property name="lift_higher_link_iyz" value="-0.00000776" scope="parent"/>
+      <xacro:property name="lift_higher_link_izz" value="0.12537280" scope="parent"/>
       <xacro:property name="higher_to_top_origin_z" value="0.2525"/>
       <xacro:property name="top_mass_value" value="1.718423"/>
       <xacro:property name="top_box_size" value="0.200 0.220 0.015"/>
-      <xacro:property name="lift_top_link_ixx" value="5.819538E-03" scope="parent"/>
-      <xacro:property name="lift_top_link_ixy" value="4.555714E-09" scope="parent"/>
-      <xacro:property name="lift_top_link_ixz" value="8.002694E-06" scope="parent"/>
-      <xacro:property name="lift_top_link_iyy" value="1.280362E-02" scope="parent"/>
-      <xacro:property name="lift_top_link_iyz" value="1.967468E-09" scope="parent"/>
-      <xacro:property name="lift_top_link_izz" value="7.048366E-03" scope="parent"/>
+      <xacro:property name="lift_top_link_ixx" value="0.00581954" scope="parent"/>
+      <xacro:property name="lift_top_link_ixy" value="0.0" scope="parent"/>
+      <xacro:property name="lift_top_link_ixz" value="0.00000800" scope="parent"/>
+      <xacro:property name="lift_top_link_iyy" value="0.01280362" scope="parent"/>
+      <xacro:property name="lift_top_link_iyz" value="0.0" scope="parent"/>
+      <xacro:property name="lift_top_link_izz" value="0.00704837" scope="parent"/>
       <xacro:property name="lift_tip_joint_origin_z" value="0.245"/>
     </xacro:if>
