Commit message: Modified 700m liftkit mass, inertia, and tier dimensional values to reflect accuracy. Also redid the meshes for 700 and re-uploaded. In the deploy launch file - added the full is_700 arg.

File: ewellix_liftkit_description/urdf/ewellix_lift.xacro (robot description, xacro)
@@ -29,8 +29,8 @@
       <xacro:property name="lift_base_link_iyz" value="0.0" scope="parent"/>
       <xacro:property name="lift_base_link_izz" value="0.00700317" scope="parent"/>
-      <xacro:property name="base_to_lower_origin_z" value="0.295"/>
+      <xacro:property name="base_to_lower_origin_z" value="0.2957"/>
       <xacro:property name="lower_mass_value" value="8.176405"/>
-      <xacro:property name="lower_box_size" value="0.163 0.163 0.575"/>
-      <xacro:property name="lower_mesh_filename" value="package://ewellix_liftkit_description/meshes/visual/lift_low_700mm.dae"/>
+      <xacro:property name="lower_box_size" value="0.163 0.163 0.5764"/>
+      <xacro:property name="lower_mesh_filename" value="package://ewellix_liftkit_description/meshes/visual/lift_low_700mm.stl"/>
       <xacro:property name="lift_lower_link_ixx" value="0.26551310" scope="parent"/>
       <xacro:property name="lift_lower_link_ixy" value="0.0" scope="parent"/>
@@ -39,8 +39,8 @@
       <xacro:property name="lift_lower_link_iyz" value="0.00111055" scope="parent"/>
       <xacro:property name="lift_lower_link_izz" value="0.26508300" scope="parent"/>
-      <xacro:property name="lower_to_higher_origin_z" value="0.0915"/>
+      <xacro:property name="lower_to_higher_origin_z" value="0.0068"/>
       <xacro:property name="middle_mass_value" value="6.54457"/>
-      <xacro:property name="middle_box_size" value="0.146 0.146 0.483"/>
-      <xacro:property name="middle_mesh_filename" value="package://ewellix_liftkit_description/meshes/visual/lift_mid_700mm.dae"/>
+      <xacro:property name="middle_box_size" value="0.146 0.146 0.5794"/>
+      <xacro:property name="middle_mesh_filename" value="package://ewellix_liftkit_description/meshes/visual/lift_mid_700mm.stl"/>
       <xacro:property name="lift_middle_link_ixx" value="0.20223860" scope="parent"/>
       <xacro:property name="lift_middle_link_ixy" value="0.0" scope="parent"/>
@@ -49,9 +49,9 @@
       <xacro:property name="lift_middle_link_iyz" value="0.0" scope="parent"/>
       <xacro:property name="lift_middle_link_izz" value="0.20223860" scope="parent"/>
-      <xacro:property name="middle_to_higher_origin_z" value="-0.03397"/>
+      <xacro:property name="middle_to_higher_origin_z" value="-0.0053"/>
       <xacro:property name="middle_upper_limit" value="0.351"/>
       <xacro:property name="higher_mass_value" value="6.375617"/>
-      <xacro:property name="higher_box_size" value="0.129 0.129 0.488"/>
-      <xacro:property name="higher_mesh_filename" value="package://ewellix_liftkit_description/meshes/visual/lift_high_700mm.dae"/>
+      <xacro:property name="higher_box_size" value="0.129 0.129 0.590"/>
+      <xacro:property name="higher_mesh_filename" value="package://ewellix_liftkit_description/meshes/visual/lift_high_700mm.stl"/>
       <xacro:property name="lift_higher_link_ixx" value="0.20932400" scope="parent"/>
       <xacro:property name="lift_higher_link_ixy" value="-0.00002260" scope="parent"/>
@@ -60,5 +60,5 @@
       <xacro:property name="lift_higher_link_iyz" value="-0.00000940" scope="parent"/>
       <xacro:property name="lift_higher_link_izz" value="0.20932130" scope="parent"/>
-      <xacro:property name="higher_to_top_origin_z" value="0.2515"/>
+      <xacro:property name="higher_to_top_origin_z" value="0.3025"/>
       <xacro:property name="top_mass_value" value="1.718423"/>
       <xacro:property name="top_box_size" value="0.200 0.220 0.015"/>
@@ -69,5 +69,5 @@
       <xacro:property name="lift_top_link_iyz" value="0.00000000" scope="parent"/>
       <xacro:property name="lift_top_link_izz" value="0.00704837" scope="parent"/>
-      <xacro:property name="lift_tip_joint_origin_z" value="0.244"/>
+      <xacro:property name="lift_tip_joint_origin_z" value="0.295"/>
     </xacro:if>
     <!--For 500 mm stroke-->

Commit message: Reverted back to all former values and meshes for the 700 mm.

File: ewellix_liftkit_description/urdf/ewellix_lift.xacro (robot description, xacro)
@@ -23,51 +23,51 @@
       <xacro:property name="base_mass_value" value="1.7383784"/>
       <xacro:property name="base_box_size" value="0.220 0.200 0.015"/>
-      <xacro:property name="lift_base_link_ixx" value="0.00577887" scope="parent"/>
+      <xacro:property name="lift_base_link_ixx" value="0.0057788770" scope="parent"/>
       <xacro:property name="lift_base_link_ixy" value="0.0" scope="parent"/>
       <xacro:property name="lift_base_link_ixz" value="0.0" scope="parent"/>
-      <xacro:property name="lift_base_link_iyy" value="0.01271701" scope="parent"/>
+      <xacro:property name="lift_base_link_iyy" value="0.0070031715" scope="parent"/>
       <xacro:property name="lift_base_link_iyz" value="0.0" scope="parent"/>
-      <xacro:property name="lift_base_link_izz" value="0.00700317" scope="parent"/>
-      <xacro:property name="base_to_lower_origin_z" value="0.2957"/>
-      <xacro:property name="lower_mass_value" value="8.176405"/>
-      <xacro:property name="lower_box_size" value="0.163 0.163 0.5764"/>
-      <xacro:property name="lower_mesh_filename" value="package://ewellix_liftkit_description/meshes/visual/lift_low_700mm.stl"/>
-      <xacro:property name="lift_lower_link_ixx" value="0.26551310" scope="parent"/>
+      <xacro:property name="lift_base_link_izz" value="0.0127170180" scope="parent"/>
+      <xacro:property name="base_to_lower_origin_z" value="0.295"/>
+      <xacro:property name="lower_mass_value" value="19.521070"/>
+      <xacro:property name="lower_box_size" value="0.163 0.163 0.575"/>
+      <xacro:property name="lower_mesh_filename" value="package://ewellix_liftkit_description/meshes/visual/lift_low_700mm.dae"/>
+      <xacro:property name="lift_lower_link_ixx" value="0.46604111" scope="parent"/>
       <xacro:property name="lift_lower_link_ixy" value="0.0" scope="parent"/>
       <xacro:property name="lift_lower_link_ixz" value="0.0" scope="parent"/>
-      <xacro:property name="lift_lower_link_iyy" value="0.06547122" scope="parent"/>
-      <xacro:property name="lift_lower_link_iyz" value="0.00111055" scope="parent"/>
-      <xacro:property name="lift_lower_link_izz" value="0.26508300" scope="parent"/>
-      <xacro:property name="lower_to_higher_origin_z" value="0.0068"/>
-      <xacro:property name="middle_mass_value" value="6.54457"/>
-      <xacro:property name="middle_box_size" value="0.146 0.146 0.5794"/>
-      <xacro:property name="middle_mesh_filename" value="package://ewellix_liftkit_description/meshes/visual/lift_mid_700mm.stl"/>
-      <xacro:property name="lift_middle_link_ixx" value="0.20223860" scope="parent"/>
+      <xacro:property name="lift_lower_link_iyy" value="0.46480515" scope="parent"/>
+      <xacro:property name="lift_lower_link_iyz" value="-0.002668667" scope="parent"/>
+      <xacro:property name="lift_lower_link_izz" value="0.1561" scope="parent"/>
+      <xacro:property name="lower_to_higher_origin_z" value="0.0915"/>
+      <xacro:property name="middle_mass_value" value="15.593303"/>
+      <xacro:property name="middle_box_size" value="0.146 0.146 0.483"/>
+      <xacro:property name="middle_mesh_filename" value="package://ewellix_liftkit_description/meshes/visual/lift_mid_700mm.dae"/>
+      <xacro:property name="lift_middle_link_ixx" value="0.34930648" scope="parent"/>
       <xacro:property name="lift_middle_link_ixy" value="0.0" scope="parent"/>
       <xacro:property name="lift_middle_link_ixz" value="0.0" scope="parent"/>
-      <xacro:property name="lift_middle_link_iyy" value="0.04003302" scope="parent"/>
+      <xacro:property name="lift_middle_link_iyy" value="0.34930648" scope="parent"/>
       <xacro:property name="lift_middle_link_iyz" value="0.0" scope="parent"/>
-      <xacro:property name="lift_middle_link_izz" value="0.20223860" scope="parent"/>
-      <xacro:property name="middle_to_higher_origin_z" value="-0.0053"/>
+      <xacro:property name="lift_middle_link_izz" value="0.095393471" scope="parent"/>
+      <xacro:property name="middle_to_higher_origin_z" value="-0.03397"/>
       <xacro:property name="middle_upper_limit" value="0.351"/>
-      <xacro:property name="higher_mass_value" value="6.375617"/>
-      <xacro:property name="higher_box_size" value="0.129 0.129 0.590"/>
-      <xacro:property name="higher_mesh_filename" value="package://ewellix_liftkit_description/meshes/visual/lift_high_700mm.stl"/>
-      <xacro:property name="lift_higher_link_ixx" value="0.20932400" scope="parent"/>
-      <xacro:property name="lift_higher_link_ixy" value="-0.00002260" scope="parent"/>
-      <xacro:property name="lift_higher_link_ixz" value="0.00000337" scope="parent"/>
-      <xacro:property name="lift_higher_link_iyy" value="0.02950402" scope="parent"/>
-      <xacro:property name="lift_higher_link_iyz" value="-0.00000940" scope="parent"/>
-      <xacro:property name="lift_higher_link_izz" value="0.20932130" scope="parent"/>
-      <xacro:property name="higher_to_top_origin_z" value="0.3025"/>
-      <xacro:property name="top_mass_value" value="1.718423"/>
+      <xacro:property name="higher_mass_value" value="15.166778"/>
+      <xacro:property name="higher_box_size" value="0.129 0.129 0.488"/>
+      <xacro:property name="higher_mesh_filename" value="package://ewellix_liftkit_description/meshes/visual/lift_high_700mm.dae"/>
+      <xacro:property name="lift_higher_link_ixx" value="0.35552099" scope="parent"/>
+      <xacro:property name="lift_higher_link_ixy" value="0.000009631" scope="parent"/>
+      <xacro:property name="lift_higher_link_ixz" value="0.000022848" scope="parent"/>
+      <xacro:property name="lift_higher_link_iyy" value="0.35552876" scope="parent"/>
+      <xacro:property name="lift_higher_link_iyz" value="0.000054910" scope="parent"/>
+      <xacro:property name="lift_higher_link_izz" value="0.069925583" scope="parent"/>
+      <xacro:property name="higher_to_top_origin_z" value="0.2515"/>
+      <xacro:property name="top_mass_value" value="4.9139525"/>
       <xacro:property name="top_box_size" value="0.200 0.220 0.015"/>
-      <xacro:property name="lift_top_link_ixx" value="0.00581954" scope="parent"/>
-      <xacro:property name="lift_top_link_ixy" value="0.00000000" scope="parent"/>
-      <xacro:property name="lift_top_link_ixz" value="0.00000800" scope="parent"/>
-      <xacro:property name="lift_top_link_iyy" value="0.01280362" scope="parent"/>
-      <xacro:property name="lift_top_link_iyz" value="0.00000000" scope="parent"/>
-      <xacro:property name="lift_top_link_izz" value="0.00704837" scope="parent"/>
-      <xacro:property name="lift_tip_joint_origin_z" value="0.295"/>
+      <xacro:property name="lift_top_link_ixx" value="0.02015548" scope="parent"/>
+      <xacro:property name="lift_top_link_ixy" value="-0.000022811" scope="parent"/>
+      <xacro:property name="lift_top_link_ixz" value="0.0" scope="parent"/>
+      <xacro:property name="lift_top_link_iyy" value="0.01664141" scope="parent"/>
+      <xacro:property name="lift_top_link_iyz" value="0.0" scope="parent"/>
+      <xacro:property name="lift_top_link_izz" value="0.03661307" scope="parent"/>
+      <xacro:property name="lift_tip_joint_origin_z" value="0.244"/>
     </xacro:if>
     <!--For 500 mm stroke-->

Commit message: Changed the 500 mm lifkit inertia values to the accurate ones. These vals worked with Gazebo.

File: ewellix_liftkit_description/urdf/ewellix_lift.xacro (robot description, xacro)
@@ -79,30 +79,30 @@
       <xacro:property name="base_mass_value" value="1.7383784"/>
       <xacro:property name="base_box_size" value="0.220 0.200 0.015"/>
-      <xacro:property name="lift_base_link_ixx" value="0.00577887" scope="parent"/>
-      <xacro:property name="lift_base_link_ixy" value="0.0" scope="parent"/>
-      <xacro:property name="lift_base_link_ixz" value="0.0" scope="parent"/>
-      <xacro:property name="lift_base_link_iyy" value="0.01271701" scope="parent"/>
-      <xacro:property name="lift_base_link_iyz" value="0.0" scope="parent"/>
-      <xacro:property name="lift_base_link_izz" value="0.00700317" scope="parent"/>
+      <xacro:property name="lift_base_link_ixx" value="0.0057788774" scope="parent"/>
+      <xacro:property name="lift_base_link_ixy" value="0" scope="parent"/>
+      <xacro:property name="lift_base_link_ixz" value="0" scope="parent"/>
+      <xacro:property name="lift_base_link_iyy" value="0.0070031719" scope="parent"/>
+      <xacro:property name="lift_base_link_iyz" value="0" scope="parent"/>
+      <xacro:property name="lift_base_link_izz" value="0.012717018" scope="parent"/>
       <xacro:property name="base_to_lower_origin_z" value="0.2457"/>
       <xacro:property name="lower_mass_value" value="6.746306"/>
       <xacro:property name="lower_box_size" value="0.163 0.163 0.4764"/>
       <xacro:property name="lower_mesh_filename" value="package://ewellix_liftkit_description/meshes/visual/lift_low_500mm.stl"/>
-      <xacro:property name="lift_lower_link_ixx" value="0.00000016" scope="parent"/>
-      <xacro:property name="lift_lower_link_ixy" value="0.0" scope="parent"/>
-      <xacro:property name="lift_lower_link_ixz" value="0.0" scope="parent"/>
-      <xacro:property name="lift_lower_link_iyy" value="0.00000005" scope="parent"/>
-      <xacro:property name="lift_lower_link_iyz" value="0.0" scope="parent"/>
-      <xacro:property name="lift_lower_link_izz" value="0.00000016" scope="parent"/>
+      <xacro:property name="lift_lower_link_ixx" value="0.1579129" scope="parent"/>
+      <xacro:property name="lift_lower_link_ixy" value="0" scope="parent"/>
+      <xacro:property name="lift_lower_link_ixz" value="0" scope="parent"/>
+      <xacro:property name="lift_lower_link_iyy" value="0.1578582" scope="parent"/>
+      <xacro:property name="lift_lower_link_iyz" value="0" scope="parent"/>
+      <xacro:property name="lift_lower_link_izz" value="0.053799503" scope="parent"/>
       <xacro:property name="lower_to_higher_origin_z" value="0.0068"/>
       <xacro:property name="middle_mass_value" value="5.411604"/>
       <xacro:property name="middle_box_size" value="0.146 0.146 0.4794"/>
       <xacro:property name="middle_mesh_filename" value="package://ewellix_liftkit_description/meshes/visual/lift_mid_500mm.stl"/>
-      <xacro:property name="lift_middle_link_ixx" value="0.11962710" scope="parent"/>
-      <xacro:property name="lift_middle_link_ixy" value="0.0" scope="parent"/>
-      <xacro:property name="lift_middle_link_ixz" value="0.0" scope="parent"/>
-      <xacro:property name="lift_middle_link_iyy" value="0.03309969" scope="parent"/>
-      <xacro:property name="lift_middle_link_iyz" value="0.0" scope="parent"/>
-      <xacro:property name="lift_middle_link_izz" value="0.11962710" scope="parent"/>
+      <xacro:property name="lift_middle_link_ixx" value="0.11963018" scope="parent"/>
+      <xacro:property name="lift_middle_link_ixy" value="0" scope="parent"/>
+      <xacro:property name="lift_middle_link_ixz" value="0" scope="parent"/>
+      <xacro:property name="lift_middle_link_iyy" value="0.11963018" scope="parent"/>
+      <xacro:property name="lift_middle_link_iyz" value="0" scope="parent"/>
+      <xacro:property name="lift_middle_link_izz" value="0.033099694" scope="parent"/>
       <xacro:property name="middle_to_higher_origin_z" value="-0.0053"/>
       <xacro:property name="middle_upper_limit" value="0.25"/>
@@ -110,19 +110,19 @@
       <xacro:property name="higher_box_size" value="0.129 0.129 0.490"/>
       <xacro:property name="higher_mesh_filename" value="package://ewellix_liftkit_description/meshes/visual/lift_high_500mm.stl"/>
-      <xacro:property name="lift_higher_link_ixx" value="0.12537550" scope="parent"/>
-      <xacro:property name="lift_higher_link_ixy" value="-0.00001864" scope="parent"/>
-      <xacro:property name="lift_higher_link_ixz" value="0.00000337" scope="parent"/>
-      <xacro:property name="lift_higher_link_iyy" value="0.02455221" scope="parent"/>
-      <xacro:property name="lift_higher_link_iyz" value="-0.00000776" scope="parent"/>
-      <xacro:property name="lift_higher_link_izz" value="0.12537280" scope="parent"/>
+      <xacro:property name="lift_higher_link_ixx" value="0.12572077" scope="parent"/>
+      <xacro:property name="lift_higher_link_ixy" value="0" scope="parent"/>
+      <xacro:property name="lift_higher_link_ixz" value="0" scope="parent"/>
+      <xacro:property name="lift_higher_link_iyy" value="0.12571806" scope="parent"/>
+      <xacro:property name="lift_higher_link_iyz" value="0" scope="parent"/>
+      <xacro:property name="lift_higher_link_izz" value="0.024552208" scope="parent"/>
       <xacro:property name="higher_to_top_origin_z" value="0.2525"/>
       <xacro:property name="top_mass_value" value="1.718423"/>
       <xacro:property name="top_box_size" value="0.200 0.220 0.015"/>
-      <xacro:property name="lift_top_link_ixx" value="0.00581954" scope="parent"/>
+      <xacro:property name="lift_top_link_ixx" value="0.0058195514" scope="parent"/>
       <xacro:property name="lift_top_link_ixy" value="0.0" scope="parent"/>
       <xacro:property name="lift_top_link_ixz" value="0.00000800" scope="parent"/>
-      <xacro:property name="lift_top_link_iyy" value="0.01280362" scope="parent"/>
+      <xacro:property name="lift_top_link_iyy" value="0.0070484261" scope="parent"/>
       <xacro:property name="lift_top_link_iyz" value="0.0" scope="parent"/>
-      <xacro:property name="lift_top_link_izz" value="0.00704837" scope="parent"/>
+      <xacro:property name="lift_top_link_izz" value="0.012803695" scope="parent"/>
       <xacro:property name="lift_tip_joint_origin_z" value="0.245"/>
     </xacro:if>
@@ -146,5 +146,5 @@
             <box size="${base_box_size}"/>
           </geometry>
-          <material name="gray"/>Home
+          <material name="gray"/>
         </visual>
         <collision>
