Commit message: Simplified liftkit to gazebo add-ons. Main changes include xacro args in urdf(s) and ros2 control addition. Rest is back to humble-devel.

File: ewellix_liftkit_description/urdf/ewellix_lift.xacro (robot description, xacro)
@@ -61,5 +61,5 @@
       <xacro:property name="lift_higher_link_iyz" value="0.000054910" scope="parent"/>
       <xacro:property name="lift_higher_link_izz" value="0.069925583" scope="parent"/>
-      <!-- <xacro:property name="higher_to_top_origin_z" value="0.2515"/>
+      <xacro:property name="higher_to_top_origin_z" value="0.2515"/>
       <xacro:property name="top_mass_value" value="4.9139525"/>
       <xacro:property name="top_box_size" value="0.200 0.220 0.015"/>
@@ -70,5 +70,5 @@
       <xacro:property name="lift_top_link_iyz" value="0.0" scope="parent"/>
       <xacro:property name="lift_top_link_izz" value="0.03661307" scope="parent"/>
-      <xacro:property name="lift_tip_joint_origin_z" value="0.244"/> -->
+      <xacro:property name="lift_tip_joint_origin_z" value="0.244"/>
     </xacro:if>
     <!--For 500 mm stroke-->
@@ -87,5 +87,4 @@
       <xacro:property name="lift_base_link_izz" value="0.012717018" scope="parent"/>
       <xacro:property name="base_to_lower_origin_z" value="0.2457"/>
-      <!-- <xacro:property name="base_to_lower_origin_z" value="0.015"/> -->
       <xacro:property name="lower_mass_value" value="6.746306"/>
       <xacro:property name="lower_box_size" value="0.163 0.163 0.4764"/>
@@ -118,6 +117,6 @@
       <xacro:property name="lift_higher_link_iyz" value="0" scope="parent"/>
       <xacro:property name="lift_higher_link_izz" value="0.024552208" scope="parent"/>
-      <!-- <xacro:property name="higher_to_top_origin_z" value="0.2525"/> -->
-      <!-- <xacro:property name="top_mass_value" value="1.718423"/>
+      <xacro:property name="higher_to_top_origin_z" value="0.2525"/>
+      <xacro:property name="top_mass_value" value="1.718423"/>
       <xacro:property name="top_box_size" value="0.200 0.220 0.015"/>
       <xacro:property name="lift_top_link_ixx" value="0.0058195514" scope="parent"/>
@@ -127,5 +126,5 @@
       <xacro:property name="lift_top_link_iyz" value="0.0" scope="parent"/>
       <xacro:property name="lift_top_link_izz" value="0.012803695" scope="parent"/>
-      <xacro:property name="lift_tip_joint_origin_z" value="0.245"/> -->
+      <xacro:property name="lift_tip_joint_origin_z" value="0.245"/>
     </xacro:if>
   <xacro:unless value="${not omit_plates}">
@@ -165,6 +164,5 @@
       <visual>
         <geometry>
-          <!-- <mesh filename= "${lower_mesh_filename}"/> -->
-          <box size="${lower_box_size}"/>
+          <mesh filename= "${lower_mesh_filename}"/>
         </geometry>
         <material name="gray"/>
@@ -192,6 +190,5 @@
       <visual>
         <geometry>
-          <!-- <mesh filename= "${middle_mesh_filename}"/> -->
-          <box size="${middle_box_size}"/>
+          <mesh filename= "${middle_mesh_filename}"/>
         </geometry>
         <material name="gray"/>
@@ -211,6 +208,5 @@
       <visual>
         <geometry>
-          <!-- <mesh filename= "${higher_mesh_filename}"/> -->
-          <box size="${higher_box_size}"/>
+          <mesh filename= "${higher_mesh_filename}"/>
         </geometry>
         <material name="gray"/>
@@ -238,4 +234,38 @@
       <limit lower="0" upper="${middle_upper_limit}" effort="1000" velocity="1"/>
       <mimic joint="${tf_prefix}ewellix_lift_lower_to_higher" multiplier="0.5" offset="0"/>
+    </joint>
+     <!--TOP (omit_plates=false)-->
+    <xacro:if value="${not omit_plates}">
+      <link name="${tf_prefix}ewellix_lift_top_link">
+        <inertia>
+          <mass value="${top_mass_value}"/>
+          <inertia ixx="${lift_top_link_ixx}" ixy="${lift_top_link_ixy}" ixz="${lift_top_link_ixz}" iyy="${lift_top_link_iyy}" iyz="${lift_top_link_iyz}" izz="${lift_top_link_izz}"/>
+        </inertia>
+        <visual>
+          <geometry>
+            <box size="${top_box_size}"/>
+          </geometry>
+          <material name="gray"/>
+        </visual>
+        <collision>
+          <geometry>
+            <box size="${top_box_size}"/>
+          </geometry>
+        </collision>
+      </link>
+    </xacro:if>
+    <!--HIGHER TO TOP (FIXED, omit_plates=false)-->
+    <xacro:if value="${not omit_plates}">
+      <joint name="${tf_prefix}higher_to_top" type="fixed">
+        <parent link="${tf_prefix}ewellix_lift_higher_link"/>
+        <child link="${tf_prefix}ewellix_lift_top_link"/>
+        <origin xyz="0 0 ${higher_to_top_origin_z}" rpy="0 0 0"/>
+      </joint>
+    </xacro:if>
+    <link name="${tf_prefix}ewellix_lift_tip_link"/>
+    <joint name="${tf_prefix}ewellix_lift_tip_joint" type="fixed">
+      <parent link="${tf_prefix}ewellix_lift_higher_link"/>
+      <child link="${tf_prefix}ewellix_lift_tip_link"/>
+      <origin xyz="0 0 ${lift_tip_joint_origin_z}" rpy="0 0 0"/>
     </joint>
     <xacro:include filename="$(find ewellix_liftkit_description)/urdf/ewellix_liftkit.ros2_control.xacro" />

File: ewellix_liftkit_description/urdf/ewellix_liftkit.ros2_control.xacro (robot description, xacro)
@@ -44,5 +44,5 @@
       </ros2_control>
     </xacro:if>
-    <!-- FOR LAUNCHING GAZEBO - Simplified LINKAGE SYSTEM -->
+    <!-- FOR LAUNCHING GAZEBO -->
     <xacro:if value="${use_gazebo}">
       <ros2_control name="${name}" type="system">
@@ -68,17 +68,4 @@
           </joint>
       </ros2_control>
-      <gazebo>
-        <plugin filename="libign_ros2_control-system.so" name="ign_ros2_control::IgnitionROS2ControlPlugin">
-          <parameters>$(find ewellix_liftkit_deploy)/config/liftkit_controllers.yaml</parameters>
-        </plugin>
-      </gazebo>
-      <gazebo>
-        <plugin filename="libignition-gazebo-pose-publisher-system.so" name="ignition::gazebo::systems::PosePublisher">
-          <publish_link_pose>true</publish_link_pose>
-          <publish_nested_model_pose>true</publish_nested_model_pose>
-          <use_pose_vector_msg>true</use_pose_vector_msg>
-          <update_frequency>50</update_frequency>
-        </plugin>
-      </gazebo>
     </xacro:if>
   </xacro:macro>

Commit message: Make ros2_control tag generation optional

File: ewellix_liftkit_description/urdf/ewellix_lift.xacro (robot description, xacro)
@@ -12,4 +12,5 @@
     com_port:=/dev/ttyUSB0
     use_gazebo:=false
+    generate_ros2_control_tag=true
     *origin
   ">
@@ -199,4 +200,8 @@
         </geometry>
       </collision>
+      <inertial>
+          <mass value="0.1"/>
+          <inertia ixx="0.01" ixy="0.0" ixz="0.0" iyy="0.01" iyz="0.0" izz="0.01"/>
+      </inertial>
     </link>
     <!--HIGHER-->
@@ -269,13 +274,15 @@
       <origin xyz="0 0 ${lift_tip_joint_origin_z}" rpy="0 0 0"/>
     </joint>
-    <xacro:include filename="$(find ewellix_liftkit_description)/urdf/ewellix_liftkit.ros2_control.xacro" />
-    <xacro:ewellix_liftkit_ros2_control
-      name="${name}"
-      use_fake_hardware="${use_fake_hardware}"
-      tf_prefix="${tf_prefix}"
-      com_port="${com_port}"
-      height_limit="${height_limit}"
-      use_gazebo="${use_gazebo}"
-    />
+    <xacro:if value="${generate_ros2_control_tag}">
+      <xacro:include filename="$(find ewellix_liftkit_description)/urdf/ewellix_liftkit.ros2_control.xacro" />
+      <xacro:ewellix_liftkit_ros2_control
+        name="${name}"
+        use_fake_hardware="${use_fake_hardware}"
+        use_gazebo="${use_gazebo}"
+        tf_prefix="${tf_prefix}"
+        com_port="${com_port}"
+        height_limit="${height_limit}"
+      />
+    </xacro:if>
   </xacro:macro>
 </robot>

Commit message: Remove redundant change after rebase

File: ewellix_liftkit_description/urdf/ewellix_lift.xacro (robot description, xacro)
@@ -200,8 +200,4 @@
         </geometry>
       </collision>
-      <inertial>
-          <mass value="0.1"/>
-          <inertia ixx="0.01" ixy="0.0" ixz="0.0" iyy="0.01" iyz="0.0" izz="0.01"/>
-      </inertial>
     </link>
     <!--HIGHER-->

Commit message: fixing 500 mm default location

File: ewellix_liftkit_description/urdf/ewellix_lift.xacro (robot description, xacro)
@@ -97,5 +97,5 @@
       <xacro:property name="lift_lower_link_iyz" value="0.0" scope="parent"/>
       <xacro:property name="lift_lower_link_izz" value="0.00000016" scope="parent"/>
-      <xacro:property name="lower_to_higher_origin_z" value="0.0068"/>
+      <xacro:property name="lower_to_higher_origin_z" value="0.0368"/>
       <xacro:property name="middle_mass_value" value="5.411604"/>
       <xacro:property name="middle_box_size" value="0.146 0.146 0.4794"/>
@@ -107,5 +107,5 @@
       <xacro:property name="lift_middle_link_iyz" value="0.0" scope="parent"/>
       <xacro:property name="lift_middle_link_izz" value="0.11962710" scope="parent"/>
-      <xacro:property name="middle_to_higher_origin_z" value="-0.0053"/>
+      <xacro:property name="middle_to_higher_origin_z" value="-0.0303"/>
       <xacro:property name="middle_upper_limit" value="0.25"/>
       <xacro:property name="higher_mass_value" value="5.324879"/>
